Commit message: added ros2_control plugin to define hardware interfaces

File: src/rushbott_common/rushbott_description/urdf/common_properties.urdf.xacro (robot description, xacro)
@@ -1,58 +1,58 @@
-<?xml version="1.0"?>
-<robot xmlns:xacro="http://www.ros.org/wiki/xacro">
+<?xml version='1.0'?>
+<robot xmlns:xacro='http://www.ros.org/wiki/xacro'>
     <!-- Inertial blocks -->
-    <xacro:macro name="inertial_cuboid_with_pose" params="mass x y z *origin">
+    <xacro:macro name='inertial_cuboid_with_pose' params='mass x y z *origin'>
         <inertial>
-            <mass value="${mass}" />
-            <xacro:insert_block name="origin"/>
-            <inertia ixx="${(1/12) * mass * (y*y + z*z)}" ixy="0.0" ixz="0.0"
-            iyy="${(1/12) * mass * (x*x + z*z)}" iyz="0.0"
-            izz="${(1/12) * mass * (x*x + y*y)}" />
+            <mass value='${mass}' />
+            <xacro:insert_block name='origin'/>
+            <inertia ixx='${(1/12) * mass * (y*y + z*z)}' ixy='0.0' ixz='0.0'
+            iyy='${(1/12) * mass * (x*x + z*z)}' iyz='0.0'
+            izz='${(1/12) * mass * (x*x + y*y)}' />
         </inertial>
     </xacro:macro>
-    <xacro:macro name="inertial_cuboid" params="mass x y z">
-        <xacro:inertial_cuboid_with_pose mass="${mass}" x="${x}" y="${y}" z="${z}">
-            <origin xyz="0 0 0" />
+    <xacro:macro name='inertial_cuboid' params='mass x y z'>
+        <xacro:inertial_cuboid_with_pose mass='${mass}' x='${x}' y='${y}' z='${z}'>
+            <origin xyz='0 0 0' />
         </xacro:inertial_cuboid_with_pose>
     </xacro:macro>
-    <xacro:macro name="inertial_cylinder_with_pose" params="mass radius length *origin">
+    <xacro:macro name='inertial_cylinder_with_pose' params='mass radius length *origin'>
         <inertial>
-            <xacro:insert_block name="origin"/>
-            <mass value="${mass}" />
-            <inertia ixx="${(1/12) * mass * (3*radius*radius + length*length)}" ixy="0.0" ixz="0.0"
-            iyy="${(1/12) * mass * (3*radius*radius + length*length)}" iyz="0.0"
-            izz="${(1/2) * mass * (radius*radius)}" />
+            <xacro:insert_block name='origin'/>
+            <mass value='${mass}' />
+            <inertia ixx='${(1/12) * mass * (3*radius*radius + length*length)}' ixy='0.0' ixz='0.0'
+            iyy='${(1/12) * mass * (3*radius*radius + length*length)}' iyz='0.0'
+            izz='${(1/2) * mass * (radius*radius)}' />
         </inertial>
     </xacro:macro>
-    <xacro:macro name="inertial_cylinder" params="mass radius length">
-        <xacro:inertial_cylinder_with_pose mass="${mass}" radius="${radius}" length="${length}">
-            <origin xyz="0 0 0" />
+    <xacro:macro name='inertial_cylinder' params='mass radius length'>
+        <xacro:inertial_cylinder_with_pose mass='${mass}' radius='${radius}' length='${length}'>
+            <origin xyz='0 0 0' />
         </xacro:inertial_cylinder_with_pose>
     </xacro:macro>
-    <xacro:macro name="inertial_sphere" params="mass radius">
+    <xacro:macro name='inertial_sphere' params='mass radius'>
         <inertial>
-            <mass value="${mass}" />
-            <inertia ixx="${(2/5) * mass * radius * radius}" ixy="0.0" ixz="0.0"
-                        iyy="${(2/5) * mass * radius * radius}" iyz="0.0"
-                        izz="${(2/5) * mass * radius * radius}" />
+            <mass value='${mass}' />
+            <inertia ixx='${(2/5) * mass * radius * radius}' ixy='0.0' ixz='0.0'
+                        iyy='${(2/5) * mass * radius * radius}' iyz='0.0'
+                        izz='${(2/5) * mass * radius * radius}' />
         </inertial>
     </xacro:macro>
-    <xacro:macro name="inertial_dummy">
-        <xacro:inertial_cuboid mass="0.01" x="0.01" y="0.01" z="0.01"/>
+    <xacro:macro name='inertial_dummy'>
+        <xacro:inertial_cuboid mass='0.01' x='0.01' y='0.01' z='0.01'/>
     </xacro:macro>
     <!-- Conversions -->
-    <xacro:property name="cm2m"    value="${1/100.0}"/>
-    <xacro:property name="mm2m"    value="${1/1000.0}"/>
-    <xacro:property name="in2m"    value="0.0254"/>
-    <xacro:property name="deg2rad" value="${pi/180.0}"/>
+    <xacro:property name='cm2m'    value='${1/100.0}'/>
+    <xacro:property name='mm2m'    value='${1/1000.0}'/>
+    <xacro:property name='in2m'    value='0.0254'/>
+    <xacro:property name='deg2rad' value='${pi/180.0}'/>
     <!-- Material colors -->
-    <xacro:property name="material_black">
-        <material name="black">
-            <color rgba="1 1 1 1"/>
+    <xacro:property name='material_black'>
+        <material name='black'>
+            <color rgba='1 1 1 1'/>
         </material>
     </xacro:property>
-    <xacro:property name="material_cyan">
-        <material name="cyan">
-            <color rgba="0 1.0 1.0 1.0"/>
+    <xacro:property name='material_cyan'>
+        <material name='cyan'>
+            <color rgba='0 1.0 1.0 1.0'/>
         </material>
     </xacro:property>

File: src/rushbott_common/rushbott_description/urdf/rushbott.urdf.xacro (robot description, xacro)
@@ -1,52 +1,58 @@
-<?xml version="1.0"?>
-<robot xmlns:xacro="http://www.ros.org/wiki/xacro" name="rushbott">
-    <xacro:include filename="common_properties.urdf.xacro"/>
-    <xacro:include filename="wheel.urdf.xacro"/>
+<?xml version='1.0'?>
+<robot xmlns:xacro='http://www.ros.org/wiki/xacro' name='rushbott'>
+    <xacro:include filename='common_properties.urdf.xacro'/>
+    <xacro:include filename='wheel.urdf.xacro'/>
     <!-- Mechanical properties -->
-    <xacro:property name="body_mass"               value="2.300" />
-    <xacro:property name="body_length"             value="${40*cm2m}" />
-    <xacro:property name="body_width"              value="${20*cm2m}" />
-    <xacro:property name="body_height"             value="${10*cm2m}" />
-    <xacro:property name="wheel_depth"            value="${body_height*(1/2)}" />
-    <xacro:property name="track_width"             value="${body_width*(3/4)}" />
-    <xacro:property name="wheelbase"               value="${body_length*(3/4)}" />
-    <xacro:property name="base_link_z_offset"      value="${15*cm2m}"/>
+    <xacro:property name='body_mass'               value='2.300' />
+    <xacro:property name='body_length'             value='${40*cm2m}' />
+    <xacro:property name='body_width'              value='${20*cm2m}' />
+    <xacro:property name='body_height'             value='${10*cm2m}' />
+    <xacro:property name='wheel_depth'            value='${body_height*(1/2)}' />
+    <xacro:property name='track_width'             value='${body_width*(3/4)}' />
+    <xacro:property name='wheelbase'               value='${body_length*(3/4)}' />
+    <xacro:property name='base_link_z_offset'      value='${15*cm2m}'/>
     <!-- Dummy link -->
-    <link name="base_footprint"/>
+    <link name='base_footprint'/>
     <!-- Base link -->
-    <joint name="base_footprint_to_base_link=" type="fixed">
-        <parent link="base_footprint"/>
-        <child link="base_link"/>
+    <joint name='base_footprint_to_base_link' type='fixed'>
+        <parent link='base_footprint'/>
+        <child link='base_link'/>
     </joint>
-    <link name="base_link">
+    <link name='base_link'>
         <visual>
-            <origin xyz="0 0 ${base_link_z_offset}" rpy="0 0 0"/>
+            <origin xyz='0 0 ${base_link_z_offset}' rpy='0 0 0'/>
             <geometry>
-                <box size="${body_length} ${body_width} ${body_height}"/>
+                <box size='${body_length} ${body_width} ${body_height}'/>
             </geometry>
-            <xacro:insert_block name="material_cyan"/>
+            <xacro:insert_block name='material_cyan'/>
         </visual>
-        <collision name="create3_base_collision">
-            <origin xyz="0 0 ${base_link_z_offset}" rpy="0 0 0"/>
+        <collision name='create3_base_collision'>
+            <origin xyz='0 0 ${base_link_z_offset}' rpy='0 0 0'/>
             <geometry>
-                <box size="${body_length} ${body_width} ${body_height}"/>
+                <box size='${body_length} ${body_width} ${body_height}'/>
             </geometry>
         </collision>
-        <xacro:inertial_cuboid_with_pose mass="${body_mass}" x="${body_length}" y="${body_width}" z="${body_height}">
-            <origin xyz="0 0 ${base_link_z_offset}"/>
+        <xacro:inertial_cuboid_with_pose mass='${body_mass}' x='${body_length}' y='${body_width}' z='${body_height}'>
+            <origin xyz='0 0 ${base_link_z_offset}'/>
         </xacro:inertial_cuboid_with_pose>
     </link>
     <!-- Wheels -->
-    <xacro:wheel name="fl_wheel" parent_link="base_link">
-        <origin xyz="${wheelbase/2} ${track_width/2} ${base_link_z_offset-wheel_depth}" rpy="${pi/2} 0 0"/>
+    <xacro:wheel name='fl_wheel' parent_link='base_link' motor='true' min_vel=-10 max_vel=10>
+        <origin xyz='${wheelbase/2} ${track_width/2} ${base_link_z_offset-wheel_depth}' rpy='${pi/2} 0 0'/>
     </xacro:wheel>
-    <xacro:wheel name="fr_wheel" parent_link="base_link">
-        <origin xyz="${wheelbase/2} ${-track_width/2} ${base_link_z_offset-wheel_depth}" rpy="${pi/2} 0 0"/>
+    <xacro:wheel name='fr_wheel' parent_link='base_link' motor='true' min_vel=-10 max_vel=10>
+        <origin xyz='${wheelbase/2} ${-track_width/2} ${base_link_z_offset-wheel_depth}' rpy='${pi/2} 0 0'/>
     </xacro:wheel>
-    <xacro:wheel name="rl_wheel" parent_link="base_link">
-        <origin xyz="${-wheelbase/2} ${track_width/2} ${base_link_z_offset-wheel_depth}" rpy="${pi/2} 0 0"/>
+    <xacro:wheel name='rl_wheel' parent_link='base_link'>
+        <origin xyz='${-wheelbase/2} ${track_width/2} ${base_link_z_offset-wheel_depth}' rpy='${pi/2} 0 0'/>
     </xacro:wheel>
-    <xacro:wheel name="rr_wheel" parent_link="base_link">
-        <origin xyz="${-wheelbase/2} ${-track_width/2} ${base_link_z_offset-wheel_depth}" rpy="${pi/2} 0 0"/>
+    <xacro:wheel name='rr_wheel' parent_link='base_link'>
+        <origin xyz='${-wheelbase/2} ${-track_width/2} ${base_link_z_offset-wheel_depth}' rpy='${pi/2} 0 0'/>
     </xacro:wheel>
+    <!-- Gazebo THIS WAS THE LAST THING U WERE DOING, U WERE ADDING THE PLUGIN TO CONNECT GAZEBO TO YOUR HARDWARE-->
+    <gazebo>
+        <plugin name='gazebo_ros2_control' filename='libgazebo_ros2_control.so'>
+            <parameters></parameters>
+        </plugin>
+    </gazebo>
 </robot>

File: src/rushbott_common/rushbott_description/urdf/wheel.urdf.xacro (robot description, xacro)
@@ -1,31 +1,46 @@
-<?xml version="1.0"?>
-<robot xmlns:xacro="http://www.ros.org/wiki/xacro">
-<xacro:macro name="wheel" params="name parent_link *origin">
-    <xacro:property name="mass"   value="0.2" />
-    <xacro:property name="radius" value="${4*cm2m}" />
-    <xacro:property name="width"  value="${2*cm2m}" />
-    <xacro:property name="wheel_link_name"  value="${name}_wheel"/>
-    <xacro:property name="wheel_joint_name" value="${wheel_link_name}_joint"/>
-    <joint name="${wheel_joint_name}" type="continuous">
-        <parent link="${parent_link}"/>
-        <child link="${wheel_link_name}"/>
-        <xacro:insert_block name="origin"/>
-        <axis xyz="0 0 1"/>
+<?xml version='1.0'?>
+<robot xmlns:xacro='http://www.ros.org/wiki/xacro'>
+<xacro:macro name='wheel' params='name parent_link *origin' 'motor="false" *min_vel *max_vel'>
+    <xacro:property name='mass'   value='0.2' />
+    <xacro:property name='radius' value='${4*cm2m}' />
+    <xacro:property name='width'  value='${2*cm2m}' />
+    <xacro:property name='wheel_link_name'  value='${name}_wheel'/>
+    <xacro:property name='wheel_joint_name' value='${wheel_link_name}_joint'/>
+    <joint name='${wheel_joint_name}' type='continuous'>
+        <parent link='${parent_link}'/>
+        <child link='${wheel_link_name}'/>
+        <xacro:insert_block name='origin'/>
+        <axis xyz='0 0 1'/>
     </joint>
-    <link name="${wheel_link_name}">
+    <link name='${wheel_link_name}'>
         <visual>
             <geometry>
-                <cylinder length="${width}" radius="${radius}"/>
+                <cylinder length='${width}' radius='${radius}'/>
             </geometry>
-            <xacro:insert_block name="material_black"/>
+            <xacro:insert_block name='material_black'/>
         </visual>
         <collision>
             <geometry>
-                <cylinder length="${width}" radius="${radius}"/>
+                <cylinder length='${width}' radius='${radius}'/>
             </geometry>
         </collision>
-        <xacro:inertial_cylinder mass="${mass}" radius="${radius}"
-            length="${width}"/>
+        <xacro:inertial_cylinder mass='${mass}' radius='${radius}'
+            length='${width}'/>
     </link>
+    <xacro:if value='${motor == "true"}'>
+        <ros2_control name='${wheel_link_name}_controller' type='system'>
+            <hardware>
+                <plugin> gazebo_ros2_control/GazeboSystem </plugin>
+            </hardware>
+            <joint name='${wheel_joint_name}'>
+                <command_interface name='velocity'>
+                    <param name='min'> ${min_vel} </param>
+                    <param name='max'> ${min_vel} </param>
+                </command_interface>
+                <state_interface name='velocity'/>
+                <state_interface name='position'/>
+            </joint>
+        </ros2_control>
+    </xacro:if>
 </xacro:macro>
 </robot>

Commit message: controllers succesfully activate

File: src/rushbott_common/rushbott_description/urdf/common_properties.urdf.xacro (robot description, xacro)
@@ -49,10 +49,20 @@
     <xacro:property name='material_black'>
         <material name='black'>
-            <color rgba='1 1 1 1'/>
+            <color rgba='0 0 0 1'/>
+        </material>
+    </xacro:property>
+    <xacro:property name='material_red'>
+        <material name='red'>
+            <color rgba='1 0 0 1'/>
         </material>
     </xacro:property>
     <xacro:property name='material_cyan'>
         <material name='cyan'>
-            <color rgba='0 1.0 1.0 1.0'/>
+            <color rgba='0 1 1 1'/>
+        </material>
+    </xacro:property>
+    <xacro:property name='material_white'>
+        <material name='white'>
+            <color rgba='1 1 1 1'/>
         </material>
     </xacro:property>

File: src/rushbott_common/rushbott_description/urdf/rushbott.urdf.xacro (robot description, xacro)
@@ -38,21 +38,21 @@
     </link>
     <!-- Wheels -->
-    <xacro:wheel name='fl_wheel' parent_link='base_link' motor='true' min_vel='-10' max_vel='10'>
+    <xacro:wheel name='fl' parent_link='base_link' motor='True' min_vel='-10' max_vel='10'>
         <origin xyz='${wheelbase/2} ${track_width/2} ${base_link_z_offset-wheel_depth}' rpy='${pi/2} 0 0'/>
     </xacro:wheel>
-    <xacro:wheel name='fr_wheel' parent_link='base_link' motor='true' min_vel='-10' max_vel='10'>
+    <xacro:wheel name='fr' parent_link='base_link' motor='True' min_vel='-10' max_vel='10'>
         <origin xyz='${wheelbase/2} ${-track_width/2} ${base_link_z_offset-wheel_depth}' rpy='${pi/2} 0 0'/>
     </xacro:wheel>
-    <xacro:wheel name='rl_wheel' parent_link='base_link'>
+    <xacro:wheel name='rl' parent_link='base_link'>
         <origin xyz='${-wheelbase/2} ${track_width/2} ${base_link_z_offset-wheel_depth}' rpy='${pi/2} 0 0'/>
     </xacro:wheel>
-    <xacro:wheel name='rr_wheel' parent_link='base_link'>
+    <xacro:wheel name='rr' parent_link='base_link'>
         <origin xyz='${-wheelbase/2} ${-track_width/2} ${base_link_z_offset-wheel_depth}' rpy='${pi/2} 0 0'/>
     </xacro:wheel>
     <!-- Gazebo (make this conditional later on)-->
-    <!-- <gazebo>
-        <plugin name='gz_ros2_control::GazeboSimROS2ControlPlugin' filename='libgz_ros2_control-system.so'>
+    <gazebo>
+        <plugin filename="libgz_ros2_control-system.so" name="gz_ros2_control::GazeboSimROS2ControlPlugin">
             <parameters>$(find rushbott_control)/config/control.yaml</parameters>
         </plugin>
-    </gazebo> -->
+    </gazebo>
 </robot>

File: src/rushbott_common/rushbott_description/urdf/wheel.urdf.xacro (robot description, xacro)
@@ -1,8 +1,16 @@
 <?xml version='1.0'?>
 <robot xmlns:xacro='http://www.ros.org/wiki/xacro'>
-<xacro:macro name='wheel' params='name parent_link *origin motor:="false" min_vel:="0" max_vel:="0"'>
+<xacro:macro name='wheel' params='name parent_link motor:=False min_vel:=0 max_vel:=0 *origin'>
     <xacro:property name='mass'   value='0.2' />
     <xacro:property name='radius' value='${4*cm2m}' />
     <xacro:property name='width'  value='${2*cm2m}' />
+    <xacro:property name='material_block'>
+        <xacro:insert_block name='material_white'/>
+    </xacro:property>
+    <xacro:if value='${motor == True}' >
+        <xacro:property name='material_block'>
+            <xacro:insert_block name='material_red'/>
+        </xacro:property>
+    </xacro:if>
     <xacro:property name='wheel_link_name'  value='${name}_wheel'/>
     <xacro:property name='wheel_joint_name' value='${wheel_link_name}_joint'/>
@@ -18,5 +26,5 @@
                 <cylinder length='${width}' radius='${radius}'/>
             </geometry>
-            <xacro:insert_block name='material_black'/>
+            <xacro:insert_block name='material_block'/>
         </visual>
         <collision>
@@ -28,13 +36,13 @@
             length='${width}'/>
     </link>
-    <xacro:if value='${motor == "true"}'>
+    <xacro:if value='${motor == True}'>
         <ros2_control name='${wheel_link_name}_controller' type='system'>
             <hardware>
-                <plugin> gz_ros2_control/GazeboSimSystem </plugin>
+                <plugin>gz_ros2_control/GazeboSimSystem</plugin>
             </hardware>
             <joint name='${wheel_joint_name}'>
                 <command_interface name='velocity'>
-                    <param name='min'> ${min_vel} </param>
-                    <param name='max'> ${min_vel} </param>
+                    <param name='min'>${min_vel}</param>
+                    <param name='max'>${min_vel}</param>
                 </command_interface>
                 <state_interface name='velocity'/>

Commit message: added arm.urdf and upperarm.urdf

File: src/rushbott_common/rushbott_description/urdf/common_properties.urdf.xacro (robot description, xacro)
@@ -62,4 +62,14 @@
         </material>
     </xacro:property>
+    <xacro:property name = "material_orange">
+        <material name="orange">
+            <color rgba="1.0 0.65 0.0 1.0"/>
+        </material>
+    </xacro:property>
+    <xacro:property name = "material_pink">
+        <material name="pink">
+            <color rgba="1.0 0.75 0.8 1.0"/>
+        </material>
+    </xacro:property>
     <xacro:property name='material_white'>
         <material name='white'>

File: src/rushbott_common/rushbott_description/urdf/rushbott.urdf.xacro (robot description, xacro)
@@ -4,4 +4,6 @@
     <xacro:include filename='wheel.urdf.xacro'/>
     <xacro:include filename='wheel_with_servo.urdf.xacro'/>
+    <xacro:include filename="arm.urdf.xacro"/>
+    <xacro:include filename="upperarm.urdf.xacro"/>
     <!-- Mechanical properties -->
     <xacro:property name='body_mass'               value='2.300' />
@@ -19,11 +21,12 @@
     <xacro:property name='servo_width'             value='${4*cm2m}' />
     <xacro:property name='servo_depth'            value='${wheel_radius+3*cm2m}' />
+    <xacro:property name = "arm_length" value = "1"/>
+    <xacro:property name = "arm_radius" value = "0.05"/>
     <!-- Base footprint -->
     <link name='base_footprint'/>
     <!-- Base link -->
-    <joint name='base_link_joint' type='fixed'>
-        <parent link='base_footprint'/>
-        <child link='base_link'/>
-        <origin xyz='0 0 ${body_height/2}'/>
+    <joint name="base_footprint_to_base_link" type="fixed">
+        <parent link="base_footprint"/>
+        <child link="base_link"/>
     </joint>
     <link name='base_link'>
@@ -77,3 +80,12 @@
         </plugin>
     </gazebo>
+    <!-- Lower Arm -->
+    <xacro:arm name = "lower_arm" parent_link = "base_link">
+        <origin xyz = "0 0 ${base_link_z_offset}" rpy = "0 0 0"/>
+        <limit lower = "0" upper = "${pi/2}" velocity = "100" effort = "100"/>
+    </xacro:arm>
+    <!-- Upper Arm -->
+    <xacro:upperarm name = "upper_arm" parent_link = "lower_arm_link">
+        <origin xyz = "${arm_length} 0 0" rpy = "0 0 0"/>
+    </xacro:upperarm>
 </robot>
