Commit message: removed joint_state_publisher, fixed update rate issues

File: src/rushbott_common/rushbott_description/urdf/wheel_with_servo.urdf.xacro (robot description, xacro)
@@ -8,9 +8,10 @@
             <xacro:insert_block name='material_red'/>
         </xacro:property>
-        <joint name='${servo_joint_name}' type='continuous'>
+        <joint name='${servo_joint_name}' type='revolute'>
             <parent link='${parent_link}'/>
             <child link='${servo_link_name}'/>
             <xacro:insert_block name='origin'/>
             <axis xyz='0 0 -1'/>
+            <limit lower = "${-pi/2}" upper = "${pi/2}" velocity = "100" effort = "100"/>
         </joint>
         <link name='${servo_link_name}'>
