Commit message: preparing branch for merging

File: src/rushbott_common/rushbott_description/urdf/arm_link.urdf.xacro (robot description, xacro)
@@ -2,5 +2,5 @@
 <robot xmlns:xacro='http://www.ros.org/wiki/xacro'>
     <!--Arm Link-->
-    <xacro:macro name='arm_link' params='name parent_link arm_length arm_mass *origin *limit'>
+    <xacro:macro name='arm_link' params='name parent_link arm_length mesh *origin *limit *inertial'>
         <xacro:property name='arm_link_name' value='${name}'/>
         <xacro:property name='arm_joint_name' value='${name}_joint'/>
@@ -32,5 +32,5 @@
     </xacro:macro>
     <!--Arm Link Mimic-->
-    <xacro:macro name='arm_link_mimic' params='name parent_link arm_length arm_mass *origin *limit *mimic'>
+    <xacro:macro name='arm_link_mimic' params='name parent_link arm_length mesh *origin *limit *inertial *mimic'>
         <xacro:property name='arm_link_name' value='${name}'/>
         <xacro:property name='arm_joint_name' value='${name}_joint'/>

File: src/rushbott_common/rushbott_description/urdf/rushbott.urdf.xacro (robot description, xacro)
@@ -92,5 +92,5 @@
     </gazebo>
     <!-- Arm -->
-    <xacro:arm_link name='lower_arm' parent_link='base_link' arm_length='${lower_arm_length}' arm_mass='${lower_arm_mass}'>
+    <!-- <xacro:arm_link name='lower_arm' parent_link='base_link' arm_length='${lower_arm_length}' arm_mass='${lower_arm_mass}'>
         <origin xyz='0 0 0.3' rpy='0 0 0'/>
         <limit lower='0' upper='${pi}' effort='10' velocity='10'/>
@@ -110,5 +110,5 @@
         <mimic joint='upper_control_joint' multiplier='1.0' offset='${pi}'/>
     </xacro:arm_link_mimic>
-    <!-- <xacro:arm_link name='suction_head' parent_link='upper_arm' arm_length='${suction_head_length}' arm_mass='${suction_head_mass}'>
+    <xacro:arm_link name='suction_head' parent_link='upper_arm' arm_length='${suction_head_length}' arm_mass='${suction_head_mass}'>
         <origin xyz='${upper_arm_length} 0 0' rpy='0 0 0'/>
         <limit lower='${-pi/2}' upper='${pi/2}' effort='10' velocity='10'/>
