Commit message: reorganized tree to seperate description and bringup packages

File: src/rushbott_common/rushbott_description/urdf/rushbott.urdf.xacro (robot description, xacro)
@@ -6,8 +6,9 @@
     <xacro:property name="body_mass"               value="2.300" />
     <xacro:property name="body_length"             value="${40*cm2m}" />
-    <xacro:property name="body_width"              value="${10*cm2m}" />
-    <xacro:property name="body_height"             value="${5*cm2m}" />
-    <xacro:property name="wheel_height"            value="${-2.75*cm2m}" />
-    <xacro:property name="distance_between_wheels" value="${23.3*cm2m}" />
+    <xacro:property name="body_width"              value="${20*cm2m}" />
+    <xacro:property name="body_height"             value="${10*cm2m}" />
+    <xacro:property name="wheel_depth"            value="${body_height*(1/2)}" />
+    <xacro:property name="track_width"             value="${body_width*(3/4)}" />
+    <xacro:property name="wheelbase"               value="${body_length*(3/4)}" />
     <xacro:property name="base_link_z_offset"      value="${6.42*cm2m}"/>
     <!-- Dummy link -->
@@ -37,9 +38,15 @@
     </link>
     <!-- Wheels -->
-    <xacro:wheel name="left_wheel" parent_link="base_link">
-        <origin xyz="0 ${distance_between_wheels/2} ${base_link_z_offset}" rpy="0 0 0"/>
+    <xacro:wheel name="fl_wheel" parent_link="base_link">
+        <origin xyz="${wheelbase/2} ${track_width/2} ${base_link_z_offset-wheel_depth}" rpy="${pi/2} 0 0"/>
     </xacro:wheel>
-    <xacro:wheel name="right_wheel" parent_link="base_link">
-        <origin xyz="0 ${-distance_between_wheels/2} ${base_link_z_offset}" rpy="0 0 0"/>
+    <xacro:wheel name="fr_wheel" parent_link="base_link">
+        <origin xyz="${wheelbase/2} ${-track_width/2} ${base_link_z_offset-wheel_depth}" rpy="${pi/2} 0 0"/>
+    </xacro:wheel>
+    <xacro:wheel name="rl_wheel" parent_link="base_link">
+        <origin xyz="${-wheelbase/2} ${track_width/2} ${base_link_z_offset-wheel_depth}" rpy="${pi/2} 0 0"/>
+    </xacro:wheel>
+    <xacro:wheel name="rr_wheel" parent_link="base_link">
+        <origin xyz="${-wheelbase/2} ${-track_width/2} ${base_link_z_offset-wheel_depth}" rpy="${pi/2} 0 0"/>
     </xacro:wheel>
 </robot>

File: src/rushbott_common/rushbott_description/urdf/wheel.urdf.xacro (robot description, xacro)
@@ -3,6 +3,6 @@
 <xacro:macro name="wheel" params="name parent_link *origin">
     <xacro:property name="mass"   value="0.2" />
-    <xacro:property name="radius" value="${3.575*cm2m}" />
-    <xacro:property name="width"  value="${1.5*cm2m}" />
+    <xacro:property name="radius" value="${4*cm2m}" />
+    <xacro:property name="width"  value="${2*cm2m}" />
     <xacro:property name="wheel_link_name"  value="${name}_wheel"/>
     <xacro:property name="wheel_joint_name" value="${wheel_link_name}_joint"/>

Commit message: gazebo now launches and spawns in robot!

File: src/rushbott_common/rushbott_description/urdf/rushbott.urdf.xacro (robot description, xacro)
@@ -11,5 +11,5 @@
     <xacro:property name="track_width"             value="${body_width*(3/4)}" />
     <xacro:property name="wheelbase"               value="${body_length*(3/4)}" />
-    <xacro:property name="base_link_z_offset"      value="${6.42*cm2m}"/>
+    <xacro:property name="base_link_z_offset"      value="${15*cm2m}"/>
     <!-- Dummy link -->
     <link name="base_footprint"/>

Commit message: worked on gazebo plugins

File: src/rushbott_common/rushbott_description/urdf/rushbott.urdf.xacro (robot description, xacro)
@@ -38,8 +38,8 @@
     </link>
     <!-- Wheels -->
-    <xacro:wheel name='fl_wheel' parent_link='base_link' motor='true' min_vel=-10 max_vel=10>
+    <xacro:wheel name='fl_wheel' parent_link='base_link' motor='true' min_vel='-10' max_vel='10'>
         <origin xyz='${wheelbase/2} ${track_width/2} ${base_link_z_offset-wheel_depth}' rpy='${pi/2} 0 0'/>
     </xacro:wheel>
-    <xacro:wheel name='fr_wheel' parent_link='base_link' motor='true' min_vel=-10 max_vel=10>
+    <xacro:wheel name='fr_wheel' parent_link='base_link' motor='true' min_vel='-10' max_vel='10'>
         <origin xyz='${wheelbase/2} ${-track_width/2} ${base_link_z_offset-wheel_depth}' rpy='${pi/2} 0 0'/>
     </xacro:wheel>
@@ -50,9 +50,9 @@
         <origin xyz='${-wheelbase/2} ${-track_width/2} ${base_link_z_offset-wheel_depth}' rpy='${pi/2} 0 0'/>
     </xacro:wheel>
-    <!-- Gazebo THIS WAS THE LAST THING U WERE DOING, U WERE ADDING THE PLUGIN TO CONNECT GAZEBO TO YOUR HARDWARE-->
-    <gazebo>
-        <plugin name='gazebo_ros2_control' filename='libgazebo_ros2_control.so'>
-            <parameters></parameters>
+    <!-- Gazebo (make this conditional later on)-->
+    <!-- <gazebo>
+        <plugin name='gz_ros2_control::GazeboSimROS2ControlPlugin' filename='libgz_ros2_control-system.so'>
+            <parameters>$(find rushbott_control)/config/control.yaml</parameters>
         </plugin>
-    </gazebo>
+    </gazebo> -->
 </robot>

File: src/rushbott_common/rushbott_description/urdf/wheel.urdf.xacro (robot description, xacro)
@@ -1,5 +1,5 @@
 <?xml version='1.0'?>
 <robot xmlns:xacro='http://www.ros.org/wiki/xacro'>
-<xacro:macro name='wheel' params='name parent_link *origin' 'motor="false" *min_vel *max_vel'>
+<xacro:macro name='wheel' params='name parent_link *origin motor:="false" min_vel:="0" max_vel:="0"'>
     <xacro:property name='mass'   value='0.2' />
     <xacro:property name='radius' value='${4*cm2m}' />
@@ -31,5 +31,5 @@
         <ros2_control name='${wheel_link_name}_controller' type='system'>
             <hardware>
-                <plugin> gazebo_ros2_control/GazeboSystem </plugin>
+                <plugin> gz_ros2_control/GazeboSimSystem </plugin>
             </hardware>
             <joint name='${wheel_joint_name}'>

Commit message: controller fixes

File: src/rushbott_common/rushbott_description/urdf/rushbott.urdf.xacro (robot description, xacro)
@@ -12,11 +12,5 @@
     <xacro:property name='wheelbase'               value='${body_length*(3/4)}' />
     <xacro:property name='base_link_z_offset'      value='${15*cm2m}'/>
-    <!-- Dummy link -->
-    <link name='base_footprint'/>
     <!-- Base link -->
-    <joint name='base_footprint_to_base_link' type='fixed'>
-        <parent link='base_footprint'/>
-        <child link='base_link'/>
-    </joint>
     <link name='base_link'>
         <visual>
@@ -38,8 +32,8 @@
     </link>
     <!-- Wheels -->
-    <xacro:wheel name='fl' parent_link='base_link' motor='True' min_vel='-10' max_vel='10'>
+    <xacro:wheel name='fl' parent_link='base_link' motor='True'>
         <origin xyz='${wheelbase/2} ${track_width/2} ${base_link_z_offset-wheel_depth}' rpy='${pi/2} 0 0'/>
     </xacro:wheel>
-    <xacro:wheel name='fr' parent_link='base_link' motor='True' min_vel='-10' max_vel='10'>
+    <xacro:wheel name='fr' parent_link='base_link' motor='True'>
         <origin xyz='${wheelbase/2} ${-track_width/2} ${base_link_z_offset-wheel_depth}' rpy='${pi/2} 0 0'/>
     </xacro:wheel>

File: src/rushbott_common/rushbott_description/urdf/wheel.urdf.xacro (robot description, xacro)
@@ -1,5 +1,5 @@
 <?xml version='1.0'?>
 <robot xmlns:xacro='http://www.ros.org/wiki/xacro'>
-<xacro:macro name='wheel' params='name parent_link motor:=False min_vel:=0 max_vel:=0 *origin'>
+<xacro:macro name='wheel' params='name parent_link motor:=False *origin'>
     <xacro:property name='mass'   value='0.2' />
     <xacro:property name='radius' value='${4*cm2m}' />
@@ -43,6 +43,6 @@
             <joint name='${wheel_joint_name}'>
                 <command_interface name='velocity'>
-                    <param name='min'>${min_vel}</param>
-                    <param name='max'>${min_vel}</param>
+                    <param name='min'>-10</param>
+                    <param name='max'>10</param>
                 </command_interface>
                 <state_interface name='velocity'/>

Commit message: she moves

File: src/rushbott_common/rushbott_description/urdf/rushbott.urdf.xacro (robot description, xacro)
@@ -9,11 +9,17 @@
     <xacro:property name='body_height'             value='${10*cm2m}' />
     <xacro:property name='wheel_depth'            value='${body_height*(1/2)}' />
-    <xacro:property name='track_width'             value='${body_width*(3/4)}' />
     <xacro:property name='wheelbase'               value='${body_length*(3/4)}' />
     <xacro:property name='base_link_z_offset'      value='${15*cm2m}'/>
     <!-- Base link -->
-    <link name='base_link'>
+    <link name='base_link'/>
+    <!-- Chassis link -->
+    <joint name='chassis_joint' type='fixed'>
+        <parent link='base_link'/>
+        <child link='chassis_link'/>
+        <origin xyz='${(body_length-wheelbase)/2} 0 0'/>
+    </joint>
+    <link name='chassis_link'>
         <visual>
-            <origin xyz='0 0 ${base_link_z_offset}' rpy='0 0 0'/>
+            <origin xyz='${-body_length/2} 0 ${body_height/2}'/>
             <geometry>
                 <box size='${body_length} ${body_width} ${body_height}'/>
@@ -22,5 +28,5 @@
         </visual>
         <collision name='create3_base_collision'>
-            <origin xyz='0 0 ${base_link_z_offset}' rpy='0 0 0'/>
+            <origin xyz='${-body_length/2} 0 ${body_height/2}'/>
             <geometry>
                 <box size='${body_length} ${body_width} ${body_height}'/>
@@ -28,19 +34,23 @@
         </collision>
         <xacro:inertial_cuboid_with_pose mass='${body_mass}' x='${body_length}' y='${body_width}' z='${body_height}'>
-            <origin xyz='0 0 ${base_link_z_offset}'/>
+            <origin xyz='${-body_length/2} 0 ${body_height/2}'/>
         </xacro:inertial_cuboid_with_pose>
     </link>
     <!-- Wheels -->
     <xacro:wheel name='fl' parent_link='base_link' motor='True'>
-        <origin xyz='${wheelbase/2} ${track_width/2} ${base_link_z_offset-wheel_depth}' rpy='${pi/2} 0 0'/>
+        <origin xyz='0 ${body_width/2} 0' rpy='${-pi/2} 0 0'/>
+        <axis xyz='0 0 1'/>
     </xacro:wheel>
     <xacro:wheel name='fr' parent_link='base_link' motor='True'>
-        <origin xyz='${wheelbase/2} ${-track_width/2} ${base_link_z_offset-wheel_depth}' rpy='${pi/2} 0 0'/>
+        <origin xyz='0 ${-body_width/2} 0' rpy='${pi/2} 0 0'/>
+        <axis xyz='0 0 -1'/>
     </xacro:wheel>
     <xacro:wheel name='rl' parent_link='base_link'>
-        <origin xyz='${-wheelbase/2} ${track_width/2} ${base_link_z_offset-wheel_depth}' rpy='${pi/2} 0 0'/>
+        <origin xyz='${-wheelbase} ${body_width/2} 0' rpy='${-pi/2} 0 0'/>
+        <axis xyz='0 0 1'/>
     </xacro:wheel>
     <xacro:wheel name='rr' parent_link='base_link'>
-        <origin xyz='${-wheelbase/2} ${-track_width/2} ${base_link_z_offset-wheel_depth}' rpy='${pi/2} 0 0'/>
+        <origin xyz='${-wheelbase} ${-body_width/2} 0' rpy='${pi/2} 0 0'/>
+        <axis xyz='0 0 -1'/>
     </xacro:wheel>
     <!-- Gazebo (make this conditional later on)-->

File: src/rushbott_common/rushbott_description/urdf/wheel.urdf.xacro (robot description, xacro)
@@ -1,5 +1,5 @@
 <?xml version='1.0'?>
 <robot xmlns:xacro='http://www.ros.org/wiki/xacro'>
-<xacro:macro name='wheel' params='name parent_link motor:=False *origin'>
+<xacro:macro name='wheel' params='name parent_link motor:=False *origin *axis'>
     <xacro:property name='mass'   value='0.2' />
     <xacro:property name='radius' value='${4*cm2m}' />
@@ -19,8 +19,9 @@
         <child link='${wheel_link_name}'/>
         <xacro:insert_block name='origin'/>
-        <axis xyz='0 0 1'/>
+        <xacro:insert_block name='axis'/>
     </joint>
     <link name='${wheel_link_name}'>
         <visual>
+            <origin xyz='0 0 ${width/2}'/>
             <geometry>
                 <cylinder length='${width}' radius='${radius}'/>
@@ -29,4 +30,5 @@
         </visual>
         <collision>
+            <origin xyz='0 0 ${width/2}'/>
             <geometry>
                 <cylinder length='${width}' radius='${radius}'/>

Commit message: it turns! also gpu wont work with gazebo on wls no matter what sadge

File: src/rushbott_common/rushbott_description/urdf/rushbott.urdf.xacro (robot description, xacro)
@@ -5,10 +5,9 @@
     <!-- Mechanical properties -->
     <xacro:property name='body_mass'               value='2.300' />
-    <xacro:property name='body_length'             value='${40*cm2m}' />
-    <xacro:property name='body_width'              value='${20*cm2m}' />
-    <xacro:property name='body_height'             value='${10*cm2m}' />
+    <xacro:property name='body_length'             value='${50*cm2m}' />
+    <xacro:property name='body_width'              value='${30*cm2m}' />
+    <xacro:property name='body_height'             value='${20*cm2m}' />
     <xacro:property name='wheel_depth'            value='${body_height*(1/2)}' />
     <xacro:property name='wheelbase'               value='${body_length*(3/4)}' />
-    <xacro:property name='base_link_z_offset'      value='${15*cm2m}'/>
     <!-- Base link -->
     <link name='base_link'/>
@@ -46,9 +45,9 @@
         <axis xyz='0 0 -1'/>
     </xacro:wheel>
-    <xacro:wheel name='rl' parent_link='base_link'>
+    <xacro:wheel name='rl' parent_link='base_link' motor='True'>
         <origin xyz='${-wheelbase} ${body_width/2} 0' rpy='${-pi/2} 0 0'/>
         <axis xyz='0 0 1'/>
     </xacro:wheel>
-    <xacro:wheel name='rr' parent_link='base_link'>
+    <xacro:wheel name='rr' parent_link='base_link' motor='True'>
         <origin xyz='${-wheelbase} ${-body_width/2} 0' rpy='${pi/2} 0 0'/>
         <axis xyz='0 0 -1'/>

File: src/rushbott_common/rushbott_description/urdf/wheel.urdf.xacro (robot description, xacro)
@@ -3,16 +3,39 @@
 <xacro:macro name='wheel' params='name parent_link motor:=False *origin *axis'>
     <xacro:property name='mass'   value='0.2' />
-    <xacro:property name='radius' value='${4*cm2m}' />
-    <xacro:property name='width'  value='${2*cm2m}' />
-    <xacro:property name='material_block'>
-        <xacro:insert_block name='material_white'/>
-    </xacro:property>
-    <xacro:if value='${motor == True}' >
+    <xacro:property name='radius' value='${10*cm2m}' />
+    <xacro:property name='width'  value='${4*cm2m}' />
+    <xacro:property name='wheel_link_name'  value='${name}_wheel'/>
+    <xacro:property name='wheel_joint_name' value='${wheel_link_name}_joint'/>
+    <xacro:if value='${motor == True}'>
         <xacro:property name='material_block'>
             <xacro:insert_block name='material_red'/>
         </xacro:property>
+        <gazebo reference='${wheel_link_name}'>
+            <mu1 value="0.1"/>
+            <mu2 value="0.1"/>
+        </gazebo>
+        <ros2_control name='${wheel_link_name}_controller' type='system'>
+            <hardware>
+                <plugin>gz_ros2_control/GazeboSimSystem</plugin>
+            </hardware>
+            <joint name='${wheel_joint_name}'>
+                <command_interface name='velocity'>
+                    <param name='min'>-10</param>
+                    <param name='max'>10</param>
+                </command_interface>
+                <state_interface name='velocity'/>
+                <state_interface name='position'/>
+            </joint>
+        </ros2_control>
     </xacro:if>
-    <xacro:property name='wheel_link_name'  value='${name}_wheel'/>
-    <xacro:property name='wheel_joint_name' value='${wheel_link_name}_joint'/>
+    <xacro:if value='${motor == False}'>
+        <xacro:property name='material_block'>
+            <xacro:insert_block name='material_white'/>
+        </xacro:property>
+        <gazebo reference='${wheel_link_name}'>
+            <mu1 value="0.001"/>
+            <mu2 value="0.001"/>
+        </gazebo>
+    </xacro:if>
     <joint name='${wheel_joint_name}' type='continuous'>
         <parent link='${parent_link}'/>
@@ -38,19 +61,4 @@
             length='${width}'/>
     </link>
-    <xacro:if value='${motor == True}'>
-        <ros2_control name='${wheel_link_name}_controller' type='system'>
-            <hardware>
-                <plugin>gz_ros2_control/GazeboSimSystem</plugin>
-            </hardware>
-            <joint name='${wheel_joint_name}'>
-                <command_interface name='velocity'>
-                    <param name='min'>-10</param>
-                    <param name='max'>10</param>
-                </command_interface>
-                <state_interface name='velocity'/>
-                <state_interface name='position'/>
-            </joint>
-        </ros2_control>
-    </xacro:if>
 </xacro:macro>
 </robot>

Commit message: robot now turns properly, added base_footprint as inertial frame of reference

File: src/rushbott_common/rushbott_description/urdf/rushbott.urdf.xacro (robot description, xacro)
@@ -8,17 +8,18 @@
     <xacro:property name='body_width'              value='${30*cm2m}' />
     <xacro:property name='body_height'             value='${20*cm2m}' />
+    <xacro:property name='wheel_radius'            value='${10*cm2m}' />
     <xacro:property name='wheel_depth'            value='${body_height*(1/2)}' />
     <xacro:property name='wheelbase'               value='${body_length*(3/4)}' />
+    <!-- Base footprint -->
+    <link name='base_footprint'/>
     <!-- Base link -->
-    <link name='base_link'/>
-    <!-- Chassis link -->
-    <joint name='chassis_joint' type='fixed'>
-        <parent link='base_link'/>
-        <child link='chassis_link'/>
-        <origin xyz='${(body_length-wheelbase)/2} 0 0'/>
+    <joint name='base_link_joint' type='fixed'>
+        <parent link='base_footprint'/>
+        <child link='base_link'/>
+        <origin xyz='0 0 ${wheel_radius}'/>
     </joint>
-    <link name='chassis_link'>
+    <link name='base_link'>
         <visual>
-            <origin xyz='${-body_length/2} 0 ${body_height/2}'/>
+            <origin xyz='0 0 ${body_height/2}'/>
             <geometry>
                 <box size='${body_length} ${body_width} ${body_height}'/>
@@ -27,5 +28,5 @@
         </visual>
         <collision name='create3_base_collision'>
-            <origin xyz='${-body_length/2} 0 ${body_height/2}'/>
+            <origin xyz='0 0 ${body_height/2}'/>
             <geometry>
                 <box size='${body_length} ${body_width} ${body_height}'/>
@@ -33,22 +34,22 @@
         </collision>
         <xacro:inertial_cuboid_with_pose mass='${body_mass}' x='${body_length}' y='${body_width}' z='${body_height}'>
-            <origin xyz='${-body_length/2} 0 ${body_height/2}'/>
+            <origin xyz='0 0 ${body_height/2}'/>
         </xacro:inertial_cuboid_with_pose>
     </link>
     <!-- Wheels -->
     <xacro:wheel name='fl' parent_link='base_link' motor='True'>
-        <origin xyz='0 ${body_width/2} 0' rpy='${-pi/2} 0 0'/>
+        <origin xyz='${wheelbase/2} ${body_width/2} 0' rpy='${-pi/2} 0 0'/>
         <axis xyz='0 0 1'/>
     </xacro:wheel>
     <xacro:wheel name='fr' parent_link='base_link' motor='True'>
-        <origin xyz='0 ${-body_width/2} 0' rpy='${pi/2} 0 0'/>
+        <origin xyz='${wheelbase/2} ${-body_width/2} 0' rpy='${pi/2} 0 0'/>
         <axis xyz='0 0 -1'/>
     </xacro:wheel>
     <xacro:wheel name='rl' parent_link='base_link' motor='True'>
-        <origin xyz='${-wheelbase} ${body_width/2} 0' rpy='${-pi/2} 0 0'/>
+        <origin xyz='${-wheelbase/2} ${body_width/2} 0' rpy='${-pi/2} 0 0'/>
         <axis xyz='0 0 1'/>
     </xacro:wheel>
     <xacro:wheel name='rr' parent_link='base_link' motor='True'>
-        <origin xyz='${-wheelbase} ${-body_width/2} 0' rpy='${pi/2} 0 0'/>
+        <origin xyz='${-wheelbase/2} ${-body_width/2} 0' rpy='${pi/2} 0 0'/>
         <axis xyz='0 0 -1'/>
     </xacro:wheel>

File: src/rushbott_common/rushbott_description/urdf/wheel.urdf.xacro (robot description, xacro)
@@ -3,5 +3,4 @@
 <xacro:macro name='wheel' params='name parent_link motor:=False *origin *axis'>
     <xacro:property name='mass'   value='0.2' />
-    <xacro:property name='radius' value='${10*cm2m}' />
     <xacro:property name='width'  value='${4*cm2m}' />
     <xacro:property name='wheel_link_name'  value='${name}_wheel'/>
@@ -12,6 +11,9 @@
         </xacro:property>
         <gazebo reference='${wheel_link_name}'>
-            <mu1 value="0.1"/>
-            <mu2 value="0.1"/>
+			<mu1 value="0.5"/>
+			<mu2 value="0.3"/>
+			<kp value="10000000.0"/>
+			<kd value="1.0"/>
+			<fdir1 value="1 0 0"/>
         </gazebo>
         <ros2_control name='${wheel_link_name}_controller' type='system'>
@@ -30,10 +32,13 @@
     </xacro:if>
     <xacro:if value='${motor == False}'>
-        <xacro:property name='material_block'>
+         <xacro:property name='material_block'>
             <xacro:insert_block name='material_white'/>
         </xacro:property>
-        <gazebo reference='${wheel_link_name}'>
-            <mu1 value="0.001"/>
-            <mu2 value="0.001"/>
+         <gazebo reference='${wheel_link_name}'>
+			<mu1 value="0.5"/>
+			<mu2 value="0.3"/>
+			<kp value="10000000.0"/>
+			<kd value="1.0"/>
+			<fdir1 value="1 0 0"/>
         </gazebo>
     </xacro:if>
@@ -48,5 +53,5 @@
             <origin xyz='0 0 ${width/2}'/>
             <geometry>
-                <cylinder length='${width}' radius='${radius}'/>
+                <cylinder length='${width}' radius='${wheel_radius}'/>
             </geometry>
             <xacro:insert_block name='material_block'/>
@@ -55,8 +60,8 @@
             <origin xyz='0 0 ${width/2}'/>
             <geometry>
-                <cylinder length='${width}' radius='${radius}'/>
+                <cylinder length='${width}' radius='${wheel_radius}'/>
             </geometry>
         </collision>
-        <xacro:inertial_cylinder mass='${mass}' radius='${radius}'
+        <xacro:inertial_cylinder mass='${mass}' radius='${wheel_radius}'
             length='${width}'/>
     </link>
