Commit message: added middle wheels and servos to the urdf

File: src/rushbott_common/rushbott_description/urdf/rushbott.urdf.xacro (robot description, xacro)
@@ -3,4 +3,5 @@
     <xacro:include filename='common_properties.urdf.xacro'/>
     <xacro:include filename='wheel.urdf.xacro'/>
+    <xacro:include filename='wheel_with_servo.urdf.xacro'/>
     <!-- Mechanical properties -->
     <xacro:property name='body_mass'               value='2.300' />
@@ -8,7 +9,14 @@
     <xacro:property name='body_width'              value='${30*cm2m}' />
     <xacro:property name='body_height'             value='${20*cm2m}' />
-    <xacro:property name='wheel_radius'            value='${10*cm2m}' />
-    <xacro:property name='wheel_depth'            value='${body_height*(1/2)}' />
-    <xacro:property name='wheelbase'               value='${body_length*(3/4)}' />
+    <xacro:property name='wheel_mass'              value='0.2' />
+    <xacro:property name='wheel_radius'            value='${7.5*cm2m}' />
+    <xacro:property name='wheel_width'             value='${5*cm2m}' />
+    <xacro:property name='wheel_depth'             value='${wheel_radius}' />
+    <xacro:property name='wheelbase'               value='${body_length*(4/5)}' />
+    <xacro:property name='track_width'             value='${body_width+wheel_width+3*cm2m}' />
+    <xacro:property name='servo_mass'              value='0.2' />
+    <xacro:property name='servo_radius'            value='${3*cm2m}' />
+    <xacro:property name='servo_width'             value='${4*cm2m}' />
+    <xacro:property name='servo_depth'            value='${wheel_radius+3*cm2m}' />
     <!-- Base footprint -->
     <link name='base_footprint'/>
@@ -17,5 +25,5 @@
         <parent link='base_footprint'/>
         <child link='base_link'/>
-        <origin xyz='0 0 ${wheel_radius}'/>
+        <origin xyz='0 0 ${body_height/2}'/>
     </joint>
     <link name='base_link'>
@@ -27,5 +35,5 @@
             <xacro:insert_block name='material_cyan'/>
         </visual>
-        <collision name='create3_base_collision'>
+        <collision>
             <origin xyz='0 0 ${body_height/2}'/>
             <geometry>
@@ -37,19 +45,28 @@
         </xacro:inertial_cuboid_with_pose>
     </link>
-    <!-- Wheels -->
-    <xacro:wheel name='fl' parent_link='base_link' motor='True'>
-        <origin xyz='${wheelbase/2} ${body_width/2} 0' rpy='${-pi/2} 0 0'/>
+    <!-- Wheels with servos-->
+    <xacro:wheel_with_servo name='fl' parent_link='base_link'>
+        <origin xyz='${wheelbase/2} ${track_width/2} ${-wheel_depth+servo_depth}' rpy='0 0 0'/>
+        <axis xyz='0 0 1'/>
+    </xacro:wheel_with_servo>
+    <xacro:wheel_with_servo name='fr' parent_link='base_link'>
+        <origin xyz='${wheelbase/2} ${-track_width/2} ${-wheel_depth+servo_depth}' rpy='0 0 ${pi}'/>
+        <axis xyz='0 0 -1'/>
+    </xacro:wheel_with_servo>
+    <xacro:wheel_with_servo name='rl' parent_link='base_link'>
+        <origin xyz='${-wheelbase/2} ${track_width/2} ${-wheel_depth+servo_depth}' rpy='0 0 0'/>
+        <axis xyz='0 0 1'/>
+    </xacro:wheel_with_servo>
+    <xacro:wheel_with_servo name='rr' parent_link='base_link'>
+        <origin xyz='${-wheelbase/2} ${-track_width/2} ${-wheel_depth+servo_depth}' rpy='0 0 ${pi}'/>
+        <axis xyz='0 0 -1'/>
+    </xacro:wheel_with_servo>
+    <!-- Wheels-->
+    <xacro:wheel name='l' parent_link='base_link'>
+        <origin xyz='0 ${track_width/2} ${-wheel_depth}' rpy='${-pi/2} 0 0'/>
         <axis xyz='0 0 1'/>
     </xacro:wheel>
-    <xacro:wheel name='fr' parent_link='base_link' motor='True'>
-        <origin xyz='${wheelbase/2} ${-body_width/2} 0' rpy='${pi/2} 0 0'/>
-        <axis xyz='0 0 -1'/>
-    </xacro:wheel>
-    <xacro:wheel name='rl' parent_link='base_link' motor='True'>
-        <origin xyz='${-wheelbase/2} ${body_width/2} 0' rpy='${-pi/2} 0 0'/>
-        <axis xyz='0 0 1'/>
-    </xacro:wheel>
-    <xacro:wheel name='rr' parent_link='base_link' motor='True'>
-        <origin xyz='${-wheelbase/2} ${-body_width/2} 0' rpy='${pi/2} 0 0'/>
+    <xacro:wheel name='r' parent_link='base_link'>
+        <origin xyz='0 ${-track_width/2} ${-wheel_depth}' rpy='${-pi/2} 0 ${pi}'/>
         <axis xyz='0 0 -1'/>
     </xacro:wheel>

File: src/rushbott_common/rushbott_description/urdf/wheel.urdf.xacro (robot description, xacro)
@@ -1,46 +1,10 @@
 <?xml version='1.0'?>
 <robot xmlns:xacro='http://www.ros.org/wiki/xacro'>
-<xacro:macro name='wheel' params='name parent_link motor:=False *origin *axis'>
-    <xacro:property name='mass'   value='0.2' />
-    <xacro:property name='width'  value='${4*cm2m}' />
+<xacro:macro name='wheel' params='name parent_link *origin *axis'>
     <xacro:property name='wheel_link_name'  value='${name}_wheel'/>
     <xacro:property name='wheel_joint_name' value='${wheel_link_name}_joint'/>
-    <xacro:if value='${motor == True}'>
-        <xacro:property name='material_block'>
-            <xacro:insert_block name='material_red'/>
-        </xacro:property>
-        <gazebo reference='${wheel_link_name}'>
-			<mu1 value="0.5"/>
-			<mu2 value="0.3"/>
-			<kp value="10000000.0"/>
-			<kd value="1.0"/>
-			<fdir1 value="1 0 0"/>
-        </gazebo>
-        <ros2_control name='${wheel_link_name}_controller' type='system'>
-            <hardware>
-                <plugin>gz_ros2_control/GazeboSimSystem</plugin>
-            </hardware>
-            <joint name='${wheel_joint_name}'>
-                <command_interface name='velocity'>
-                    <param name='min'>-10</param>
-                    <param name='max'>10</param>
-                </command_interface>
-                <state_interface name='velocity'/>
-                <state_interface name='position'/>
-            </joint>
-        </ros2_control>
-    </xacro:if>
-    <xacro:if value='${motor == False}'>
-         <xacro:property name='material_block'>
-            <xacro:insert_block name='material_white'/>
-        </xacro:property>
-         <gazebo reference='${wheel_link_name}'>
-			<mu1 value="0.5"/>
-			<mu2 value="0.3"/>
-			<kp value="10000000.0"/>
-			<kd value="1.0"/>
-			<fdir1 value="1 0 0"/>
-        </gazebo>
-    </xacro:if>
+    <xacro:property name='material_block'>
+        <xacro:insert_block name='material_black'/>
+    </xacro:property>
     <joint name='${wheel_joint_name}' type='continuous'>
         <parent link='${parent_link}'/>
@@ -51,19 +15,38 @@
     <link name='${wheel_link_name}'>
         <visual>
-            <origin xyz='0 0 ${width/2}'/>
+            <origin xyz='0 0 0'/>
             <geometry>
-                <cylinder length='${width}' radius='${wheel_radius}'/>
+                <cylinder length='${wheel_width}' radius='${wheel_radius}'/>
             </geometry>
             <xacro:insert_block name='material_block'/>
         </visual>
         <collision>
-            <origin xyz='0 0 ${width/2}'/>
+            <origin xyz='0 0 0'/>
             <geometry>
-                <cylinder length='${width}' radius='${wheel_radius}'/>
+                <cylinder length='${wheel_width}' radius='${wheel_radius}'/>
             </geometry>
         </collision>
-        <xacro:inertial_cylinder mass='${mass}' radius='${wheel_radius}'
-            length='${width}'/>
+        <xacro:inertial_cylinder mass='${wheel_mass}' radius='${wheel_radius}' length='${wheel_width}'/>
     </link>
+    <ros2_control name='${wheel_link_name}_controller' type='system'>
+        <hardware>
+            <plugin>gz_ros2_control/GazeboSimSystem</plugin>
+        </hardware>
+        <joint name='${wheel_joint_name}'>
+            <command_interface name='velocity'>
+                <param name='min'>-10</param>
+                <param name='max'>10</param>
+            </command_interface>
+            <state_interface name='velocity'/>
+            <state_interface name='position'/>
+        </joint>
+    </ros2_control>
+    <gazebo reference='${wheel_link_name}'>
+        <mu1 value="0.5"/>
+        <mu2 value="0.3"/>
+        <kp value="10000000.0"/>
+        <kd value="1.0"/>
+        <fdir1 value="1 0 0"/>
+    </gazebo>
 </xacro:macro>
 </robot>

Commit message: changed diffdrive to ackermannsteering

File: src/rushbott_common/rushbott_description/urdf/rushbott.urdf.xacro (robot description, xacro)
@@ -13,6 +13,6 @@
     <xacro:property name='wheel_width'             value='${5*cm2m}' />
     <xacro:property name='wheel_depth'             value='${wheel_radius}' />
-    <xacro:property name='wheelbase'               value='${body_length*(4/5)}' />
-    <xacro:property name='track_width'             value='${body_width+wheel_width+3*cm2m}' />
+    <xacro:property name='wheelbase'               value='${40*cm2m}' />
+    <xacro:property name='track_width'             value='${38*cm2m}' />
     <xacro:property name='servo_mass'              value='0.2' />
     <xacro:property name='servo_radius'            value='${3*cm2m}' />
@@ -63,9 +63,9 @@
     </xacro:wheel_with_servo>
     <!-- Wheels-->
-    <xacro:wheel name='l' parent_link='base_link'>
+    <xacro:wheel name='ml' parent_link='base_link'>
         <origin xyz='0 ${track_width/2} ${-wheel_depth}' rpy='${-pi/2} 0 0'/>
         <axis xyz='0 0 1'/>
     </xacro:wheel>
-    <xacro:wheel name='r' parent_link='base_link'>
+    <xacro:wheel name='mr' parent_link='base_link'>
         <origin xyz='0 ${-track_width/2} ${-wheel_depth}' rpy='${-pi/2} 0 ${pi}'/>
         <axis xyz='0 0 -1'/>

Commit message: updated arm.urdf and upperarm.urdf

File: src/rushbott_common/rushbott_description/urdf/rushbott.urdf.xacro (robot description, xacro)
@@ -82,5 +82,5 @@
     <!-- Lower Arm -->
     <xacro:arm name = "lower_arm" parent_link = "base_link">
-        <origin xyz = "0 0 ${base_link_z_offset}" rpy = "0 0 0"/>
+        <origin xyz = "0 0 0" rpy = "0 0 0"/>
         <limit lower = "0" upper = "${pi/2}" velocity = "100" effort = "100"/>
     </xacro:arm>

Commit message: rover controller connects to ros2_control joint controllers

File: src/rushbott_common/rushbott_description/urdf/rushbott.urdf.xacro (robot description, xacro)
@@ -20,5 +20,5 @@
     <xacro:property name='servo_radius'            value='${3*cm2m}' />
     <xacro:property name='servo_width'             value='${4*cm2m}' />
-    <xacro:property name='servo_depth'            value='${wheel_radius+3*cm2m}' />
+    <xacro:property name='servo_height'            value='${wheel_radius+3*cm2m}' />
     <xacro:property name = "arm_length" value = "1"/>
     <xacro:property name = "arm_radius" value = "0.05"/>
@@ -29,4 +29,5 @@
         <parent link="base_footprint"/>
         <child link="base_link"/>
+        <origin xyz='0 0 ${wheel_depth+wheel_radius}'/>
     </joint>
     <link name='base_link'>
@@ -50,17 +51,17 @@
     <!-- Wheels with servos-->
     <xacro:wheel_with_servo name='left_front' parent_link='base_link'>
-        <origin xyz='${wheelbase/2} ${track_width/2} ${-wheel_depth+servo_depth}' rpy='0 0 0'/>
+        <origin xyz='${wheelbase/2} ${track_width/2} ${-wheel_depth+servo_height}' rpy='0 0 0'/>
         <axis xyz='0 0 1'/>
     </xacro:wheel_with_servo>
     <xacro:wheel_with_servo name='right_front' parent_link='base_link'>
-        <origin xyz='${wheelbase/2} ${-track_width/2} ${-wheel_depth+servo_depth}' rpy='0 0 ${pi}'/>
+        <origin xyz='${wheelbase/2} ${-track_width/2} ${-wheel_depth+servo_height}' rpy='0 0 ${pi}'/>
         <axis xyz='0 0 -1'/>
     </xacro:wheel_with_servo>
     <xacro:wheel_with_servo name='left_rear' parent_link='base_link'>
-        <origin xyz='${-wheelbase/2} ${track_width/2} ${-wheel_depth+servo_depth}' rpy='0 0 0'/>
+        <origin xyz='${-wheelbase/2} ${track_width/2} ${-wheel_depth+servo_height}' rpy='0 0 0'/>
         <axis xyz='0 0 1'/>
     </xacro:wheel_with_servo>
     <xacro:wheel_with_servo name='right_rear' parent_link='base_link'>
-        <origin xyz='${-wheelbase/2} ${-track_width/2} ${-wheel_depth+servo_depth}' rpy='0 0 ${pi}'/>
+        <origin xyz='${-wheelbase/2} ${-track_width/2} ${-wheel_depth+servo_height}' rpy='0 0 ${pi}'/>
         <axis xyz='0 0 -1'/>
     </xacro:wheel_with_servo>
@@ -80,12 +81,12 @@
         </plugin>
     </gazebo>
-    <!-- Lower Arm -->
+    <!-- Lower Arm
     <xacro:arm name = "lower_arm" parent_link = "base_link">
         <origin xyz = "0 0 0" rpy = "0 0 0"/>
         <limit lower = "0" upper = "${pi/2}" velocity = "100" effort = "100"/>
-    </xacro:arm>
-    <!-- Upper Arm -->
+    </xacro:arm> -->
+    <!-- Upper Arm
     <xacro:upperarm name = "upper_arm" parent_link = "lower_arm_link">
         <origin xyz = "${arm_length} 0 0" rpy = "0 0 0"/>
-    </xacro:upperarm>
+    </xacro:upperarm>  -->
 </robot>

File: src/rushbott_common/rushbott_description/urdf/wheel.urdf.xacro (robot description, xacro)
@@ -29,5 +29,5 @@
         <xacro:inertial_cylinder mass='${wheel_mass}' radius='${wheel_radius}' length='${wheel_width}'/>
     </link>
-    <ros2_control name='GazeboSystem' type='system'>
+    <ros2_control name='${wheel_joint_name}' type='system'>
         <hardware>
             <plugin>gz_ros2_control/GazeboSimSystem</plugin>

File: src/rushbott_common/rushbott_description/urdf/wheel_with_servo.urdf.xacro (robot description, xacro)
@@ -12,5 +12,5 @@
             <child link='${servo_link_name}'/>
             <xacro:insert_block name='origin'/>
-            <xacro:insert_block name='axis'/>
+            <axis xyz='0 0 -1'/>
         </joint>
         <link name='${servo_link_name}'>
@@ -30,6 +30,14 @@
             <xacro:inertial_cylinder mass='${servo_mass}' radius='${servo_radius}' length='${servo_width}'/>
         </link>
+        <ros2_control name='${servo_joint_name}' type='system'>
+            <hardware>
+                <plugin>gz_ros2_control/GazeboSimSystem</plugin>
+            </hardware>
+            <joint name='${servo_joint_name}'>
+                <command_interface name='position'/>
+            </joint>
+        </ros2_control>
         <xacro:wheel name='${name}' parent_link='${servo_link_name}'>
-            <origin xyz='0 0 ${-servo_depth}' rpy='${-pi/2} 0 0'/>
+            <origin xyz='0 0 ${-servo_height}' rpy='${-pi/2} 0 0'/>
             <xacro:insert_block name='axis'/>
         </xacro:wheel>

Commit message: more urdf fixing, adding moveit2 stuff

File: src/rushbott_common/rushbott_description/urdf/rushbott.urdf.xacro (robot description, xacro)
@@ -4,6 +4,5 @@
     <xacro:include filename='wheel.urdf.xacro'/>
     <xacro:include filename='wheel_with_servo.urdf.xacro'/>
-    <xacro:include filename="arm.urdf.xacro"/>
-    <xacro:include filename="upperarm.urdf.xacro"/>
+    <xacro:include filename='arm_link.urdf.xacro'/>
     <!-- Mechanical properties -->
     <xacro:property name='body_mass'               value='2.300' />
@@ -21,12 +20,23 @@
     <xacro:property name='servo_width'             value='${4*cm2m}' />
     <xacro:property name='servo_height'            value='${wheel_radius+3*cm2m}' />
-    <xacro:property name = "arm_length" value = "1"/>
-    <xacro:property name = "arm_radius" value = "0.05"/>
+    <xacro:property name='lower_arm_length'        value='${50*cm2m}'/>
+    <xacro:property name='lower_arm_mass'          value='0.05'/>
+    <xacro:property name='upper_control_length'    value='${20*cm2m}'/>
+    <xacro:property name='upper_control_mass'      value='0.05'/>
+    <xacro:property name='upper_link_length'       value='${lower_arm_length}'/>
+    <xacro:property name='upper_link_mass'         value='0.05'/>
+    <xacro:property name='upper_arm_length'        value='${100*cm2m}'/>
+    <xacro:property name='upper_arm_mass'          value='0.05'/>
+    <xacro:property name='suction_head_length'     value='${5*cm2m}'/>
+    <xacro:property name='suction_head_mass'       value='0.05'/>
+    <xacro:property name='arm_radius'              value='${2*cm2m}'/>
+    <xacro:property name='arm_x_position'          value='${2*cm2m}'/>
+    <xacro:property name='arm_y_position'          value='${2*cm2m}'/>
     <!-- Base footprint -->
     <link name='base_footprint'/>
     <!-- Base link -->
-    <joint name="base_footprint_to_base_link" type="fixed">
-        <parent link="base_footprint"/>
-        <child link="base_link"/>
+    <joint name='base_footprint_to_base_link' type='fixed'>
+        <parent link='base_footprint'/>
+        <child link='base_link'/>
         <origin xyz='0 0 ${wheel_depth+wheel_radius}'/>
     </joint>
@@ -77,16 +87,30 @@
     <!-- Gazebo (make this conditional later on)-->
     <gazebo>
-        <plugin filename="libgz_ros2_control-system.so" name="gz_ros2_control::GazeboSimROS2ControlPlugin">
+        <plugin filename='libgz_ros2_control-system.so' name='gz_ros2_control::GazeboSimROS2ControlPlugin'>
             <parameters>$(find rushbott_control)/config/control.yaml</parameters>
         </plugin>
     </gazebo>
-    <!-- Lower Arm
-    <xacro:arm name = "lower_arm" parent_link = "base_link">
-        <origin xyz = "0 0 0" rpy = "0 0 0"/>
-        <limit lower = "0" upper = "${pi/2}"/>
-    </xacro:arm> -->
-    <!-- Upper Arm
-    <xacro:upperarm name = "upper_arm" parent_link = "lower_arm_link">
-        <origin xyz = "${arm_length} 0 0" rpy = "0 0 0"/>
-    </xacro:upperarm>  -->
+    <!-- Arm -->
+    <xacro:arm_link name='lower_arm' parent_link='base_link' arm_length='${lower_arm_length}' arm_mass='${lower_arm_mass}'>
+        <origin xyz='0 0 0.3' rpy='0 0 0'/>
+        <limit lower='0' upper='${pi}' effort='10' velocity='10'/>
+    </xacro:arm_link>
+    <xacro:arm_link name='upper_control' parent_link='lower_arm' arm_length='${upper_control_length}' arm_mass='${upper_control_mass}'>
+        <origin xyz='0 0 0' rpy='0 0 0'/>
+        <limit lower='${-pi/2}' upper='${pi/2}' effort='10' velocity='10'/>
+    </xacro:arm_link>
+    <xacro:arm_link_mimic name='upper_link' parent_link='upper_control' arm_length='${lower_arm_length}' arm_mass='${upper_link_mass}'>
+        <origin xyz='${-upper_control_length} 0 0' rpy='0 0 0'/>
+        <limit lower='${-pi/2}' upper='${pi/2}' effort='10' velocity='10'/>
+        <mimic joint='upper_control_joint' multiplier='-1.0'/>
+    </xacro:arm_link_mimic>
+    <xacro:arm_link_mimic name='upper_arm' parent_link='upper_link' arm_length='${lower_arm_length}' arm_mass='${upper_arm_mass}'>
+        <origin xyz='${-upper_link_length} 0 0' rpy='0 0 0'/>
+        <limit lower='${-pi/2}' upper='${pi/2}' effort='10' velocity='10'/>
+        <mimic joint='upper_control_joint' multiplier='1.0' offset='${pi}'/>
+    </xacro:arm_link_mimic>
+    <!-- <xacro:arm_link name='suction_head' parent_link='upper_arm' arm_length='${suction_head_length}' arm_mass='${suction_head_mass}'>
+        <origin xyz='${upper_arm_length} 0 0' rpy='0 0 0'/>
+        <limit lower='${-pi/2}' upper='${pi/2}' effort='10' velocity='10'/>
+    </xacro:arm_link> -->
 </robot>

File: src/rushbott_common/rushbott_description/urdf/wheel_with_servo.urdf.xacro (robot description, xacro)
@@ -13,5 +13,5 @@
             <xacro:insert_block name='origin'/>
             <axis xyz='0 0 -1'/>
-            <limit lower = "${-pi/2}" upper = "${pi/2}" velocity = "10"/>
+            <limit lower = "${-pi/2}" upper = "${pi/2}" effort='10' velocity='10'/>
         </joint>
         <link name='${servo_link_name}'>

Commit message: gazebo lasers working

File: src/rushbott_common/rushbott_description/urdf/rushbott.urdf.xacro (robot description, xacro)
@@ -6,4 +6,5 @@
     <xacro:include filename="arm.urdf.xacro"/>
     <xacro:include filename="upperarm.urdf.xacro"/>
+    <xacro:include filename="lidar.urdf.xacro"/>
     <!-- Mechanical properties -->
     <xacro:property name='body_mass'               value='2.300' />
@@ -89,3 +90,7 @@
         <origin xyz = "${arm_length} 0 0" rpy = "0 0 0"/>
     </xacro:upperarm>
+    <!-- Lidar -->
+    <xacro:lidar name="lidar" parent_link="base_footprint">
+        <origin xyz="0.122 0 ${body_height}" rpy="0 0 0"/>
+    </xacro:lidar>
 </robot>

Commit message: fixed lidar after merge

File: src/rushbott_common/rushbott_description/urdf/rushbott.urdf.xacro (robot description, xacro)
@@ -114,3 +114,7 @@
         <limit lower='${-pi/2}' upper='${pi/2}' effort='10' velocity='10'/>
     </xacro:arm_link> -->
+    <!-- Lidar -->
+    <xacro:lidar parent_link="base_link">
+        <origin xyz="0.122 0 ${body_height}" rpy="0 0 0"/>
+    </xacro:lidar>
 </robot>

Commit message: moveit2 config is working

File: src/rushbott_common/rushbott_description/urdf/rushbott.urdf.xacro (robot description, xacro)
@@ -113,17 +113,17 @@
         <limit lower='${-pi}' upper='${pi}' effort='10' velocity='10'/>
     </xacro:arm_link>
-    <xacro:arm_link name='upper_control' parent_link='lower_arm' length='${upper_control_length}' width='${upper_control_width}' mass='${upper_control_mass}' mesh='${upper_control_mesh}'>
+    <xacro:arm_link name='upper_arm' parent_link='lower_arm' length='${upper_arm_length}' width='${upper_arm_width}' mass='${upper_arm_mass}' mesh='${upper_arm_mesh}'>
+        <origin xyz='${-lower_arm_length} 0 0' rpy='0 ${pi} 0'/>
+        <limit lower='${-pi}' upper='${pi}' effort='10' velocity='10'/>
+    </xacro:arm_link>
+    <xacro:arm_link_mimic name='upper_control' parent_link='lower_arm' length='${upper_control_length}' width='${upper_control_width}' mass='${upper_control_mass}' mesh='${upper_control_mesh}'>
         <origin xyz='0 0 0' rpy='0 0 0'/>
         <limit lower='${-pi}' upper='0' effort='10' velocity='10'/>
-    </xacro:arm_link>
+        <mimic joint='upper_arm_joint' multiplier='1.0'/>
+    </xacro:arm_link_mimic>
     <xacro:arm_link_mimic name='upper_link' parent_link='upper_control' length='${upper_link_length}' width='${upper_link_width}' mass='${upper_link_mass}' mesh='${upper_link_mesh}'>
         <origin xyz='${-upper_control_length} 0 0' rpy='0 0 0'/>
         <limit lower='${-pi}' upper='${pi}' effort='10' velocity='10'/>
         <mimic joint='upper_control_joint' multiplier='-1.0'/>
-    </xacro:arm_link_mimic>
-    <xacro:arm_link_mimic name='upper_arm' parent_link='upper_link' length='${upper_arm_length}' width='${upper_arm_width}' mass='${upper_arm_mass}' mesh='${upper_arm_mesh}'>
-        <origin xyz='${-upper_link_length} 0 0' rpy='0 0 0'/>
-        <limit lower='${-pi}' upper='${pi}' effort='10' velocity='10'/>
-        <mimic joint='upper_control_joint' multiplier='1.0' offset='${pi}'/>
     </xacro:arm_link_mimic>
     <xacro:arm_link name='suction_base' parent_link='upper_arm' length='${suction_base_length}' width='${suction_base_width}' mass='${suction_base_mass}' mesh='${suction_base_mesh}'>
