Commit message: changing from strings to bytes

File: src/rushbott_common/rushbott_description/urdf/rushbott.urdf.xacro (robot description, xacro)
@@ -7,5 +7,5 @@
     <xacro:include filename='lidar.urdf.xacro'/>
     <!-- Simulation Check-->
-    <xacro:property name='is_sim'               value='True' />
+    <xacro:property name='is_sim'               value='False' />
     <!-- Body Properties -->
     <xacro:property name='body_mass'               value='2.300' />
@@ -107,10 +107,10 @@
     <xacro:arm_link name='lower_arm' is_fake='false' parent_link='base_link' length='${lower_arm_length}' width='${lower_arm_width}' mass='${lower_arm_mass}' offset='0' mesh='${lower_arm_mesh}'>
         <origin xyz='${arm_x_position} 0 ${arm_z_position}' rpy='0 0 0'/>
-        <limit lower='${26 * pi / 180}' upper='${pi-0.3}' effort='10' velocity='10'/>
+        <limit lower='${-100 * 26 * pi / 180}' upper='${100 * pi-0.3}' effort='10' velocity='10'/>
     </xacro:arm_link>
     <xacro:arm_link name='upper_arm' is_fake='false' parent_link='lower_arm' length='${upper_arm_length}' width='${upper_arm_width}' mass='${upper_arm_mass}' offset='${upper_control_length}' mesh='${upper_arm_mesh}'>
         <origin xyz='${-lower_arm_length} 0 0' rpy='0 0 0'/>
-        <limit lower='${-pi+(21 * pi / 180)}' upper='${-(21 * pi / 180)}' effort='10' velocity='10'/>
-    </xacro:arm_link>w
+        <limit lower='${-pi+(21 * pi / 180) * -100}' upper='${-(21 * pi / 180) * -100}' effort='10' velocity='10'/>
+    </xacro:arm_link>
     <xacro:arm_link_mimic name='upper_control' parent_link='lower_arm' length='${upper_control_length}' width='${upper_control_width}' mass='${upper_control_mass}' mesh='${upper_control_mesh}'>
         <origin xyz='0 0 0' rpy='0 0 0'/>
@@ -140,7 +140,5 @@
                 <param name="baud_rate">9600</param>
                 <param name="msg_attempts">6</param>
-                <param name="timeout_ms">300</param>
-                <param name="stepper_lower_initial">28</param>
-                <param name="stepper_upper_initial">-28</param>
+                <param name="timeout_ms">1000</param>
                 <param name="stepper_gear_ratio">3</param>
                 <param name="stepper_enc_per_rev">400</param>
@@ -151,8 +149,10 @@
                 <command_interface name="position"/>
                 <state_interface name="position"/>
+                <param name="initial_value">-28</param>
             </joint>
             <joint name="upper_arm_joint">
                 <command_interface name="position"/>
                 <state_interface name="position"/>
+                <param name="initial_value">-28</param>
             </joint>
         </ros2_control>

Commit message: packets work, quite a bit of issues with moveit2

File: src/rushbott_common/rushbott_description/urdf/rushbott.urdf.xacro (robot description, xacro)
@@ -78,36 +78,38 @@
         </xacro:inertial_cuboid_with_pose>
     </link>
-    <!-- Wheels with servos -->
-    <xacro:wheel_with_servo name='front_left' parent_link='base_link'>
-        <origin xyz='${wheelbase/2} ${track_width/2} ${-wheel_depth+servo_height}' rpy='0 0 0'/>
-        <axis xyz='0 0 1'/>
-    </xacro:wheel_with_servo>
-    <xacro:wheel_with_servo name='front_right' parent_link='base_link'>
-        <origin xyz='${wheelbase/2} ${-track_width/2} ${-wheel_depth+servo_height}' rpy='0 0 ${pi}'/>
-        <axis xyz='0 0 -1'/>
-    </xacro:wheel_with_servo>
-    <xacro:wheel_with_servo name='rear_left' parent_link='base_link'>
-        <origin xyz='${-wheelbase/2} ${track_width/2} ${-wheel_depth+servo_height}' rpy='0 0 0'/>
-        <axis xyz='0 0 1'/>
-    </xacro:wheel_with_servo>
-    <xacro:wheel_with_servo name='rear_right' parent_link='base_link'>
-        <origin xyz='${-wheelbase/2} ${-track_width/2} ${-wheel_depth+servo_height}' rpy='0 0 ${pi}'/>
-        <axis xyz='0 0 -1'/>
-    </xacro:wheel_with_servo>
-    <!-- Wheels -->
-    <xacro:wheel name='mid_left' parent_link='base_link'>
-        <origin xyz='0 ${track_width/2} ${-wheel_depth}' rpy='${-pi/2} 0 0'/>
-        <axis xyz='0 0 1'/>
-    </xacro:wheel>
-    <xacro:wheel name='mid_right' parent_link='base_link'>
-        <origin xyz='0 ${-track_width/2} ${-wheel_depth}' rpy='${-pi/2} 0 ${pi}'/>
-        <axis xyz='0 0 -1'/>
-    </xacro:wheel>
+    <xacro:if value="${is_sim == True}">
+        <!-- Wheels with servos -->
+        <xacro:wheel_with_servo name='front_left' parent_link='base_link'>
+            <origin xyz='${wheelbase/2} ${track_width/2} ${-wheel_depth+servo_height}' rpy='0 0 0'/>
+            <axis xyz='0 0 1'/>
+        </xacro:wheel_with_servo>
+        <xacro:wheel_with_servo name='front_right' parent_link='base_link'>
+            <origin xyz='${wheelbase/2} ${-track_width/2} ${-wheel_depth+servo_height}' rpy='0 0 ${pi}'/>
+            <axis xyz='0 0 -1'/>
+        </xacro:wheel_with_servo>
+        <xacro:wheel_with_servo name='rear_left' parent_link='base_link'>
+            <origin xyz='${-wheelbase/2} ${track_width/2} ${-wheel_depth+servo_height}' rpy='0 0 0'/>
+            <axis xyz='0 0 1'/>
+        </xacro:wheel_with_servo>
+        <xacro:wheel_with_servo name='rear_right' parent_link='base_link'>
+            <origin xyz='${-wheelbase/2} ${-track_width/2} ${-wheel_depth+servo_height}' rpy='0 0 ${pi}'/>
+            <axis xyz='0 0 -1'/>
+        </xacro:wheel_with_servo>
+        <!-- Wheels -->
+        <xacro:wheel name='mid_left' parent_link='base_link'>
+            <origin xyz='0 ${track_width/2} ${-wheel_depth}' rpy='${-pi/2} 0 0'/>
+            <axis xyz='0 0 1'/>
+        </xacro:wheel>
+        <xacro:wheel name='mid_right' parent_link='base_link'>
+            <origin xyz='0 ${-track_width/2} ${-wheel_depth}' rpy='${-pi/2} 0 ${pi}'/>
+            <axis xyz='0 0 -1'/>
+        </xacro:wheel>
+    </xacro:if>
     <!-- Arm -->
-    <xacro:arm_link name='lower_arm' is_fake='false' parent_link='base_link' length='${lower_arm_length}' width='${lower_arm_width}' mass='${lower_arm_mass}' offset='0' mesh='${lower_arm_mesh}'>
+    <xacro:arm_link name='lower_arm' is_fake='true' parent_link='base_link' length='${lower_arm_length}' width='${lower_arm_width}' mass='${lower_arm_mass}' offset='0' mesh='${lower_arm_mesh}'>
         <origin xyz='${arm_x_position} 0 ${arm_z_position}' rpy='0 0 0'/>
         <limit lower='${-100 * 26 * pi / 180}' upper='${100 * pi-0.3}' effort='10' velocity='10'/>
     </xacro:arm_link>
-    <xacro:arm_link name='upper_arm' is_fake='false' parent_link='lower_arm' length='${upper_arm_length}' width='${upper_arm_width}' mass='${upper_arm_mass}' offset='${upper_control_length}' mesh='${upper_arm_mesh}'>
+    <xacro:arm_link name='upper_arm' is_fake='true' parent_link='lower_arm' length='${upper_arm_length}' width='${upper_arm_width}' mass='${upper_arm_mass}' offset='${upper_control_length}' mesh='${upper_arm_mesh}'>
         <origin xyz='${-lower_arm_length} 0 0' rpy='0 0 0'/>
         <limit lower='${-pi+(21 * pi / 180) * -100}' upper='${-(21 * pi / 180) * -100}' effort='10' velocity='10'/>
@@ -121,5 +123,5 @@
         <mimic joint='upper_control_joint' multiplier='-1.0'/>
     </xacro:arm_link_mimic>
-    <xacro:arm_link name='suction_base' is_fake='false' parent_link='upper_arm' length='${suction_base_length}' width='${suction_base_width}' mass='${suction_base_mass}' offset='0' mesh='${suction_base_mesh}'>
+    <xacro:arm_link name='suction_base' is_fake='true' parent_link='upper_arm' length='${suction_base_length}' width='${suction_base_width}' mass='${suction_base_mass}' offset='0' mesh='${suction_base_mesh}'>
         <origin xyz='${-upper_control_length+upper_arm_length} 0 0' rpy='0 0 0'/>
         <limit lower='${-2*pi}' upper='${2*pi}' effort='10' velocity='10'/>
@@ -132,4 +134,5 @@
         <origin xyz="0.122 0 ${body_height}" rpy="0 0 0"/>
     </xacro:lidar>
+    <!--
     <xacro:if value="${is_sim == False}">
         <ros2_control name="rushbott_control" type="system">
@@ -139,6 +142,6 @@
                 <param name="device">/dev/ttyACM0</param>
                 <param name="baud_rate">9600</param>
-                <param name="msg_attempts">6</param>
-                <param name="timeout_ms">1000</param>
+                <param name="msg_attempts">10</param>
+                <param name="timeout_ms">600</param>
                 <param name="stepper_gear_ratio">3</param>
                 <param name="stepper_enc_per_rev">400</param>
@@ -149,13 +152,13 @@
                 <command_interface name="position"/>
                 <state_interface name="position"/>
-                <param name="initial_value">-28</param>
+                <param name="initial_value">0.3</param>
             </joint>
             <joint name="upper_arm_joint">
                 <command_interface name="position"/>
                 <state_interface name="position"/>
-                <param name="initial_value">-28</param>
+                <param name="initial_value">-0.3</param>
             </joint>
         </ros2_control>
-    </xacro:if>
+    </xacro:if> -->
         <!-- Gazebo (make this conditional later on) -->
     <xacro:if value="${is_sim == True}">

Commit message: servo tuning

File: src/rushbott_common/rushbott_description/urdf/rushbott.urdf.xacro (robot description, xacro)
@@ -107,11 +107,11 @@
     </xacro:if>
     <!-- Arm -->
-    <xacro:arm_link name='lower_arm' is_fake='True' parent_link='base_link' length='${lower_arm_length}' width='${lower_arm_width}' mass='${lower_arm_mass}' offset='0' mesh='${lower_arm_mesh}'>
+    <xacro:arm_link name='lower_arm' is_fake='False' parent_link='base_link' length='${lower_arm_length}' width='${lower_arm_width}' mass='${lower_arm_mass}' offset='0' mesh='${lower_arm_mesh}'>
         <origin xyz='${arm_x_position} 0 ${arm_z_position}' rpy='0 0 0'/>
-        <limit lower='${-100 * 26 * pi / 180}' upper='${100 * pi-0.3}' effort='10' velocity='10'/>
+        <limit lower='${26 * pi / 180}' upper='${pi-0.3}' effort='10' velocity='10'/>
     </xacro:arm_link>
-    <xacro:arm_link name='upper_arm' is_fake='True' parent_link='lower_arm' length='${upper_arm_length}' width='${upper_arm_width}' mass='${upper_arm_mass}' offset='${upper_control_length}' mesh='${upper_arm_mesh}'>
+    <xacro:arm_link name='upper_arm' is_fake='False' parent_link='lower_arm' length='${upper_arm_length}' width='${upper_arm_width}' mass='${upper_arm_mass}' offset='${upper_control_length}' mesh='${upper_arm_mesh}'>
         <origin xyz='${-lower_arm_length} 0 0' rpy='0 0 0'/>
-        <limit lower='${-pi+(21 * pi / 180) * -100}' upper='${-(21 * pi / 180) * -100}' effort='10' velocity='10'/>
+        <limit lower='${-pi+(21 * pi / 180)}' upper='${-(21 * pi / 180)}' effort='10' velocity='10'/>
     </xacro:arm_link>
     <xacro:arm_link_mimic name='upper_control' parent_link='lower_arm' length='${upper_control_length}' width='${upper_control_width}' mass='${upper_control_mass}' mesh='${upper_control_mesh}'>
@@ -134,5 +134,4 @@
         <origin xyz="0.122 0 ${body_height}" rpy="0 0 0"/>
     </xacro:lidar>
-    <!--
     <xacro:if value="${is_sim == False}">
         <ros2_control name="rushbott_control" type="system">
@@ -160,5 +159,5 @@
             </joint>
         </ros2_control>
-    </xacro:if> -->
+    </xacro:if>
         <!-- Gazebo (make this conditional later on) -->
     <xacro:if value="${is_sim == True}">
