Commit message: moveit2

File: src/rushbott_common/rushbott_description/urdf/arm.urdf.xacro (robot description, xacro)
@@ -2,5 +2,5 @@
 <robot xmlns:xacro='http://www.ros.org/wiki/xacro'>
     <!--Arm Link-->
-    <xacro:macro name='arm_link' params='name parent_link length width mass mesh *origin *limit'>
+    <xacro:macro name='arm_link' params='name parent_link length width mass mesh initial_value *origin *limit'>
         <xacro:property name='arm_joint_name' value='${name}_joint'/>
         <joint name='${arm_joint_name}' type='revolute'>
@@ -33,5 +33,7 @@
             </hardware>
             <joint name='${arm_joint_name}'>
-                <command_interface name='position'/>
+                <command_interface name='position'>
+                    <param name="initial_value">${initial_value}</param>
+                </command_interface>
                 <state_interface name='position'/>
             </joint>

File: src/rushbott_common/rushbott_description/urdf/rushbott.urdf.xacro (robot description, xacro)
@@ -27,8 +27,10 @@
     <xacro:property name='lower_arm_width'         value='${4.5*cm2m}'/>
     <xacro:property name='lower_arm_mass'          value='0.05'/>
+    <xacro:property name='lower_arm_initial'       value='0.0'/>
     <xacro:property name='lower_arm_mesh'          value='package://rushbott_description/meshes/lower_arm.STL'/>
     <xacro:property name='upper_control_length'    value='${9.9*cm2m}'/>
     <xacro:property name='upper_control_width'     value='${2.5*cm2m}'/>
     <xacro:property name='upper_control_mass'      value='0.05'/>
+    <xacro:property name='upper_control_initial'   value='-0.5'/>
     <xacro:property name='upper_control_mesh'      value='package://rushbott_description/meshes/upper_control.STL'/>
     <xacro:property name='upper_link_length'       value='${lower_arm_length}'/>
@@ -43,4 +45,5 @@
     <xacro:property name='suction_base_width'      value='${10*cm2m}'/>
     <xacro:property name='suction_base_mass'       value='0.05'/>
+    <xacro:property name='suction_base_initial'    value='0.0'/>
     <xacro:property name='suction_base_mesh'       value='package://rushbott_description/meshes/suction_base.STL'/>
     <xacro:property name='suction_head_length'     value='${1.2*cm2m}'/>
@@ -109,9 +112,9 @@
     </gazebo>
     <!-- Arm -->
-    <xacro:arm_link name='lower_arm' parent_link='base_link' length='${lower_arm_length}' width='${lower_arm_width}' mass='${lower_arm_mass}' mesh='${lower_arm_mesh}'>
+    <xacro:arm_link name='lower_arm' parent_link='base_link' length='${lower_arm_length}' width='${lower_arm_width}' mass='${lower_arm_mass}' initial_value='${lower_arm_initial}' mesh='${lower_arm_mesh}'>
         <origin xyz='${arm_x_position} 0 ${arm_z_position}' rpy='0 0 0'/>
-        <limit lower='0' upper='${pi}' effort='10' velocity='10'/>
+        <limit lower='${-pi/2}' upper='${pi/2}' effort='10' velocity='10'/>
     </xacro:arm_link>
-    <xacro:arm_link name='upper_control' parent_link='lower_arm' length='${upper_control_length}' width='${upper_control_width}' mass='${upper_control_mass}' mesh='${upper_control_mesh}'>
+    <xacro:arm_link name='upper_control' parent_link='lower_arm' length='${upper_control_length}' width='${upper_control_width}' mass='${upper_control_mass}' initial_value='${upper_control_initial}' mesh='${upper_control_mesh}'>
         <origin xyz='0 0 0' rpy='0 0 0'/>
         <limit lower='${-pi/2}' upper='${pi/2}' effort='10' velocity='10'/>
@@ -127,5 +130,5 @@
         <mimic joint='upper_control_joint' multiplier='1.0' offset='${pi}'/>
     </xacro:arm_link_mimic>
-    <xacro:arm_link name='suction_base' parent_link='upper_arm' length='${suction_base_length}' width='${suction_base_width}' mass='${suction_base_mass}' mesh='${suction_base_mesh}'>
+    <xacro:arm_link name='suction_base' parent_link='upper_arm' length='${suction_base_length}' width='${suction_base_width}' mass='${suction_base_mass}' initial_value='${suction_base_initial}' mesh='${suction_base_mesh}'>
         <origin xyz='${-upper_arm_length} 0 0' rpy='0 0 0'/>
         <limit lower='${-pi/2}' upper='${pi/2}' effort='10' velocity='10'/>

Commit message: markers work, nothing else does this is pain

File: src/rushbott_common/rushbott_description/urdf/arm.urdf.xacro (robot description, xacro)
@@ -2,5 +2,5 @@
 <robot xmlns:xacro='http://www.ros.org/wiki/xacro'>
     <!--Arm Link-->
-    <xacro:macro name='arm_link' params='name parent_link length width mass mesh initial_value *origin *limit'>
+    <xacro:macro name='arm_link' params='name parent_link length width mass mesh *origin *limit'>
         <xacro:property name='arm_joint_name' value='${name}_joint'/>
         <joint name='${arm_joint_name}' type='revolute'>
@@ -17,4 +17,5 @@
                     <mesh filename='${mesh}' scale='0.001 0.001 0.001'/>
                 </geometry>
+                <xacro:insert_block name='material_orange'/>
             </visual>
             <collision>
@@ -33,7 +34,5 @@
             </hardware>
             <joint name='${arm_joint_name}'>
-                <command_interface name='position'>
-                    <param name="initial_value">${initial_value}</param>
-                </command_interface>
+                <command_interface name='position'/>
                 <state_interface name='position'/>
             </joint>
@@ -57,4 +56,5 @@
                     <mesh filename='${mesh}' scale='0.001 0.001 0.001'/>
                 </geometry>
+                <xacro:insert_block name='material_orange'/>
             </visual>
             <collision>
@@ -83,4 +83,5 @@
                     <mesh filename='${mesh}' scale='0.001 0.001 0.001'/>
                 </geometry>
+                <xacro:insert_block name='material_orange'/>
             </visual>
             <collision>

File: src/rushbott_common/rushbott_description/urdf/rushbott.urdf.xacro (robot description, xacro)
@@ -27,10 +27,8 @@
     <xacro:property name='lower_arm_width'         value='${4.5*cm2m}'/>
     <xacro:property name='lower_arm_mass'          value='0.05'/>
-    <xacro:property name='lower_arm_initial'       value='0.0'/>
     <xacro:property name='lower_arm_mesh'          value='package://rushbott_description/meshes/lower_arm.STL'/>
     <xacro:property name='upper_control_length'    value='${9.9*cm2m}'/>
     <xacro:property name='upper_control_width'     value='${2.5*cm2m}'/>
     <xacro:property name='upper_control_mass'      value='0.05'/>
-    <xacro:property name='upper_control_initial'   value='-0.5'/>
     <xacro:property name='upper_control_mesh'      value='package://rushbott_description/meshes/upper_control.STL'/>
     <xacro:property name='upper_link_length'       value='${lower_arm_length}'/>
@@ -45,5 +43,4 @@
     <xacro:property name='suction_base_width'      value='${10*cm2m}'/>
     <xacro:property name='suction_base_mass'       value='0.05'/>
-    <xacro:property name='suction_base_initial'    value='0.0'/>
     <xacro:property name='suction_base_mesh'       value='package://rushbott_description/meshes/suction_base.STL'/>
     <xacro:property name='suction_head_length'     value='${1.2*cm2m}'/>
@@ -112,25 +109,25 @@
     </gazebo>
     <!-- Arm -->
-    <xacro:arm_link name='lower_arm' parent_link='base_link' length='${lower_arm_length}' width='${lower_arm_width}' mass='${lower_arm_mass}' initial_value='${lower_arm_initial}' mesh='${lower_arm_mesh}'>
+    <xacro:arm_link name='lower_arm' parent_link='base_link' length='${lower_arm_length}' width='${lower_arm_width}' mass='${lower_arm_mass}' mesh='${lower_arm_mesh}'>
         <origin xyz='${arm_x_position} 0 ${arm_z_position}' rpy='0 0 0'/>
-        <limit lower='${-pi/2}' upper='${pi/2}' effort='10' velocity='10'/>
+        <limit lower='${-pi}' upper='${pi}' effort='10' velocity='10'/>
     </xacro:arm_link>
-    <xacro:arm_link name='upper_control' parent_link='lower_arm' length='${upper_control_length}' width='${upper_control_width}' mass='${upper_control_mass}' initial_value='${upper_control_initial}' mesh='${upper_control_mesh}'>
+    <xacro:arm_link name='upper_control' parent_link='lower_arm' length='${upper_control_length}' width='${upper_control_width}' mass='${upper_control_mass}' mesh='${upper_control_mesh}'>
         <origin xyz='0 0 0' rpy='0 0 0'/>
-        <limit lower='${-pi/2}' upper='${pi/2}' effort='10' velocity='10'/>
+        <limit lower='${-pi}' upper='0' effort='10' velocity='10'/>
     </xacro:arm_link>
     <xacro:arm_link_mimic name='upper_link' parent_link='upper_control' length='${upper_link_length}' width='${upper_link_width}' mass='${upper_link_mass}' mesh='${upper_link_mesh}'>
         <origin xyz='${-upper_control_length} 0 0' rpy='0 0 0'/>
-        <limit lower='${-pi/2}' upper='${pi/2}' effort='10' velocity='10'/>
+        <limit lower='${-pi}' upper='${pi}' effort='10' velocity='10'/>
         <mimic joint='upper_control_joint' multiplier='-1.0'/>
     </xacro:arm_link_mimic>
     <xacro:arm_link_mimic name='upper_arm' parent_link='upper_link' length='${upper_arm_length}' width='${upper_arm_width}' mass='${upper_arm_mass}' mesh='${upper_arm_mesh}'>
         <origin xyz='${-upper_link_length} 0 0' rpy='0 0 0'/>
-        <limit lower='${-pi/2}' upper='${pi/2}' effort='10' velocity='10'/>
+        <limit lower='${-pi}' upper='${pi}' effort='10' velocity='10'/>
         <mimic joint='upper_control_joint' multiplier='1.0' offset='${pi}'/>
     </xacro:arm_link_mimic>
-    <xacro:arm_link name='suction_base' parent_link='upper_arm' length='${suction_base_length}' width='${suction_base_width}' mass='${suction_base_mass}' initial_value='${suction_base_initial}' mesh='${suction_base_mesh}'>
+    <xacro:arm_link name='suction_base' parent_link='upper_arm' length='${suction_base_length}' width='${suction_base_width}' mass='${suction_base_mass}' mesh='${suction_base_mesh}'>
         <origin xyz='${-upper_arm_length} 0 0' rpy='0 0 0'/>
-        <limit lower='${-pi/2}' upper='${pi/2}' effort='10' velocity='10'/>
+        <limit lower='${-pi}' upper='${pi}' effort='10' velocity='10'/>
     </xacro:arm_link>
     <xacro:end_effector name='suction_head' parent_link='suction_base' length='${suction_head_length}' width='${suction_head_width}' mass='${suction_head_mass}' mesh='${suction_head_mesh}'>

File: src/rushbott_common/rushbott_description/urdf/wheel.urdf.xacro (robot description, xacro)
@@ -34,8 +34,5 @@
         </hardware>
         <joint name='${wheel_joint_name}'>
-            <command_interface name='velocity'>
-                <param name='min'>-10</param>
-                <param name='max'>10</param>
-            </command_interface>
+            <command_interface name='velocity'/>
             <state_interface name='position'/>
         </joint>

Commit message: fixed arm urdf again and changed kinematics solver Also started hardware interface development

File: src/rushbott_common/rushbott_description/urdf/arm.urdf.xacro (robot description, xacro)
@@ -2,5 +2,5 @@
 <robot xmlns:xacro='http://www.ros.org/wiki/xacro'>
     <!--Arm Link-->
-    <xacro:macro name='arm_link' params='name parent_link length width mass mesh *origin *limit'>
+    <xacro:macro name='arm_link' params='name parent_link length width offset mass mesh *origin *limit'>
         <xacro:property name='arm_joint_name' value='${name}_joint'/>
         <joint name='${arm_joint_name}' type='revolute'>
@@ -13,5 +13,5 @@
         <link name='${name}'>
             <visual>
-                <origin xyz="0 0 0" rpy="${-pi/2} 0 ${-pi/2}"/>
+                <origin xyz="0 0 0" rpy="${-pi/2} ${-pi} ${-pi/2}"/>
                 <geometry>
                     <mesh filename='${mesh}' scale='0.001 0.001 0.001'/>
@@ -20,5 +20,5 @@
             </visual>
             <collision>
-                <origin xyz='${-length/2} 0 0' rpy ='0 ${pi/2} 0'/>
+                <origin xyz='${offset-length/2} 0 0' rpy ='0 ${pi/2} 0'/>
                 <geometry>
                     <box size='${width} ${width} ${length}'/>
@@ -26,5 +26,5 @@
             </collision>
             <xacro:inertial_cuboid_with_pose mass='${mass}' x='${width}' y='${width}' z='${length}'>
-                <origin xyz='${-length/2} 0 0' rpy='0 ${pi/2} 0'/>
+                <origin xyz='${offset-length/2} 0 0' rpy='0 ${pi/2} 0'/>
             </xacro:inertial_cuboid_with_pose>
         </link>
@@ -35,4 +35,5 @@
             <joint name='${arm_joint_name}'>
                 <command_interface name='position'/>
+                    <!-- <param name='initial_value'>0.3</param> -->
                 <state_interface name='position'/>
             </joint>
@@ -40,11 +41,10 @@
     </xacro:macro>
     <!--Arm Link Mimic-->
-    <xacro:macro name='arm_link_mimic' params='name parent_link length width mass mesh *origin *limit *mimic'>
+    <xacro:macro name='arm_link_mimic' params='name parent_link length width mass mesh *origin *mimic'>
         <xacro:property name='arm_joint_name' value='${name}_joint'/>
-        <joint name='${arm_joint_name}' type='revolute'>
+        <joint name='${arm_joint_name}' type='continuous'>
             <parent link='${parent_link}'/>
             <child link='${name}'/>
             <xacro:insert_block name='origin'/>
-            <xacro:insert_block name='limit'/>
             <xacro:insert_block name='mimic'/>
             <axis xyz='0 1 0'/>
@@ -52,5 +52,5 @@
         <link name='${name}'>
             <visual>
-                <origin xyz="0 0 0" rpy="${-pi/2} 0 ${-pi/2}"/>
+                <origin xyz="0 0 0" rpy="${-pi/2} ${-pi} ${-pi/2}"/>
                 <geometry>
                     <mesh filename='${mesh}' scale='0.001 0.001 0.001'/>
@@ -79,5 +79,5 @@
         <link name='${name}'>
             <visual>
-                <origin xyz="0 0 0" rpy="${pi/2} 0 ${pi/2}"/>
+                <origin xyz="0 0 0" rpy="${-pi/2} ${-pi} ${-pi/2}"/>
                 <geometry>
                     <mesh filename='${mesh}' scale='0.001 0.001 0.001'/>

File: src/rushbott_common/rushbott_description/urdf/rushbott.urdf.xacro (robot description, xacro)
@@ -45,5 +45,5 @@
     <xacro:property name='suction_base_mesh'       value='package://rushbott_description/meshes/suction_base.STL'/>
     <xacro:property name='suction_head_length'     value='${1.2*cm2m}'/>
-    <xacro:property name='suction_head_width'      value='${16*cm2m}'/>
+    <xacro:property name='suction_head_width'      value='${10*cm2m}'/>
     <xacro:property name='suction_head_mass'       value='0.05'/>
     <xacro:property name='suction_head_mesh'       value='package://rushbott_description/meshes/suction_head.STL'/>
@@ -109,28 +109,26 @@
     </gazebo>
     <!-- Arm -->
-    <xacro:arm_link name='lower_arm' parent_link='base_link' length='${lower_arm_length}' width='${lower_arm_width}' mass='${lower_arm_mass}' mesh='${lower_arm_mesh}'>
+    <xacro:arm_link name='lower_arm' parent_link='base_link' length='${lower_arm_length}' width='${lower_arm_width}' mass='${lower_arm_mass}' offset='0' mesh='${lower_arm_mesh}'>
         <origin xyz='${arm_x_position} 0 ${arm_z_position}' rpy='0 0 0'/>
-        <limit lower='${-pi}' upper='${pi}' effort='10' velocity='10'/>
+        <limit lower='${0.3}' upper='${pi-0.3}' effort='10' velocity='10'/>
     </xacro:arm_link>
-    <xacro:arm_link name='upper_arm' parent_link='lower_arm' length='${upper_arm_length}' width='${upper_arm_width}' mass='${upper_arm_mass}' mesh='${upper_arm_mesh}'>
-        <origin xyz='${-lower_arm_length} 0 0' rpy='0 ${pi} 0'/>
-        <limit lower='${-pi}' upper='${pi}' effort='10' velocity='10'/>
+    <xacro:arm_link name='upper_arm' parent_link='lower_arm' length='${upper_arm_length}' width='${upper_arm_width}' mass='${upper_arm_mass}' offset='${upper_control_length}' mesh='${upper_arm_mesh}'>
+        <origin xyz='${-lower_arm_length} 0 0' rpy='0 0 0'/>
+        <limit lower='${-pi+0.3}' upper='${-0.3}' effort='10' velocity='10'/>
     </xacro:arm_link>
     <xacro:arm_link_mimic name='upper_control' parent_link='lower_arm' length='${upper_control_length}' width='${upper_control_width}' mass='${upper_control_mass}' mesh='${upper_control_mesh}'>
         <origin xyz='0 0 0' rpy='0 0 0'/>
-        <limit lower='${-pi}' upper='0' effort='10' velocity='10'/>
         <mimic joint='upper_arm_joint' multiplier='1.0'/>
     </xacro:arm_link_mimic>
     <xacro:arm_link_mimic name='upper_link' parent_link='upper_control' length='${upper_link_length}' width='${upper_link_width}' mass='${upper_link_mass}' mesh='${upper_link_mesh}'>
         <origin xyz='${-upper_control_length} 0 0' rpy='0 0 0'/>
-        <limit lower='${-pi}' upper='${pi}' effort='10' velocity='10'/>
         <mimic joint='upper_control_joint' multiplier='-1.0'/>
     </xacro:arm_link_mimic>
-    <xacro:arm_link name='suction_base' parent_link='upper_arm' length='${suction_base_length}' width='${suction_base_width}' mass='${suction_base_mass}' mesh='${suction_base_mesh}'>
-        <origin xyz='${-upper_arm_length} 0 0' rpy='0 0 0'/>
-        <limit lower='${-pi}' upper='${pi}' effort='10' velocity='10'/>
+    <xacro:arm_link name='suction_base' parent_link='upper_arm' length='${suction_base_length}' width='${suction_base_width}' mass='${suction_base_mass}' offset='0' mesh='${suction_base_mesh}'>
+        <origin xyz='${-upper_control_length+upper_arm_length} 0 0' rpy='0 0 0'/>
+        <limit lower='${-2*pi}' upper='${2*pi}' effort='10' velocity='10'/>
     </xacro:arm_link>
     <xacro:end_effector name='suction_head' parent_link='suction_base' length='${suction_head_length}' width='${suction_head_width}' mass='${suction_head_mass}' mesh='${suction_head_mesh}'>
-        <origin xyz='${-suction_base_length-suction_head_length} 0 0' rpy='0 0 0'/>
+        <origin xyz='${suction_base_length} 0 0' rpy='0 0 0'/>
     </xacro:end_effector>
     <!-- Lidar -->

Commit message: made rushbott hardware component

File: src/rushbott_common/rushbott_description/urdf/arm.urdf.xacro (robot description, xacro)
@@ -29,5 +29,5 @@
             </xacro:inertial_cuboid_with_pose>
         </link>
-        <ros2_control name='${arm_joint_name}' type='system'>
+        <!-- <ros2_control name='${arm_joint_name}' type='system'>
             <hardware>
                 <plugin>gz_ros2_control/GazeboSimSystem</plugin>
@@ -35,8 +35,7 @@
             <joint name='${arm_joint_name}'>
                 <command_interface name='position'/>
-                    <!-- <param name='initial_value'>0.3</param> -->
                 <state_interface name='position'/>
             </joint>
-        </ros2_control>
+        </ros2_control> -->
     </xacro:macro>
     <!--Arm Link Mimic-->

File: src/rushbott_common/rushbott_description/urdf/rushbott.urdf copy.xacro (robot description, xacro)
@@ -76,4 +76,36 @@
         </xacro:inertial_cuboid_with_pose>
     </link>
+    <!-- Wheels with servos-->
+    <xacro:wheel_with_servo name='front_left' parent_link='base_link'>
+        <origin xyz='${wheelbase/2} ${track_width/2} ${-wheel_depth+servo_height}' rpy='0 0 0'/>
+        <axis xyz='0 0 1'/>
+    </xacro:wheel_with_servo>
+    <xacro:wheel_with_servo name='front_right' parent_link='base_link'>
+        <origin xyz='${wheelbase/2} ${-track_width/2} ${-wheel_depth+servo_height}' rpy='0 0 ${pi}'/>
+        <axis xyz='0 0 -1'/>
+    </xacro:wheel_with_servo>
+    <xacro:wheel_with_servo name='rear_left' parent_link='base_link'>
+        <origin xyz='${-wheelbase/2} ${track_width/2} ${-wheel_depth+servo_height}' rpy='0 0 0'/>
+        <axis xyz='0 0 1'/>
+    </xacro:wheel_with_servo>
+    <xacro:wheel_with_servo name='rear_right' parent_link='base_link'>
+        <origin xyz='${-wheelbase/2} ${-track_width/2} ${-wheel_depth+servo_height}' rpy='0 0 ${pi}'/>
+        <axis xyz='0 0 -1'/>
+    </xacro:wheel_with_servo>
+    <!-- Wheels-->
+    <xacro:wheel name='mid_left' parent_link='base_link'>
+        <origin xyz='0 ${track_width/2} ${-wheel_depth}' rpy='${-pi/2} 0 0'/>
+        <axis xyz='0 0 1'/>
+    </xacro:wheel>
+    <xacro:wheel name='mid_right' parent_link='base_link'>
+        <origin xyz='0 ${-track_width/2} ${-wheel_depth}' rpy='${-pi/2} 0 ${pi}'/>
+        <axis xyz='0 0 -1'/>
+    </xacro:wheel>
+    <!-- Gazebo (make this conditional later on)-->
+    <gazebo>
+        <plugin filename='libgz_ros2_control-system.so' name='gz_ros2_control::GazeboSimROS2ControlPlugin'>
+            <parameters>$(find rushbott_control)/config/control.yaml</parameters>
+        </plugin>
+    </gazebo>
     <!-- Arm -->
     <xacro:arm_link name='lower_arm' parent_link='base_link' length='${lower_arm_length}' width='${lower_arm_width}' mass='${lower_arm_mass}' offset='0' mesh='${lower_arm_mesh}'>
@@ -81,5 +113,5 @@
         <limit lower='${0.3}' upper='${pi-0.3}' effort='10' velocity='10'/>
     </xacro:arm_link>
-    <!-- <xacro:arm_link name='upper_arm' parent_link='lower_arm' length='${upper_arm_length}' width='${upper_arm_width}' mass='${upper_arm_mass}' offset='${upper_control_length}' mesh='${upper_arm_mesh}'>
+    <xacro:arm_link name='upper_arm' parent_link='lower_arm' length='${upper_arm_length}' width='${upper_arm_width}' mass='${upper_arm_mass}' offset='${upper_control_length}' mesh='${upper_arm_mesh}'>
         <origin xyz='${-lower_arm_length} 0 0' rpy='0 0 0'/>
         <limit lower='${-pi+0.3}' upper='${-0.3}' effort='10' velocity='10'/>
@@ -99,19 +131,8 @@
     <xacro:end_effector name='suction_head' parent_link='suction_base' length='${suction_head_length}' width='${suction_head_width}' mass='${suction_head_mass}' mesh='${suction_head_mesh}'>
         <origin xyz='${suction_base_length} 0 0' rpy='0 0 0'/>
-    </xacro:end_effector> -->
-    <ros2_control name="rushbott_control" type="system">
-      <hardware>
-        <plugin>rushbott_hardware/RoverSystemHardware</plugin>
-        <param name="loop_rate">30</param>
-        <param name="device">/dev/serial/by-path/platform-fd500000.pcie-pci-0000:01:00.0-usb-0:1.3:1.0-port0</param>
-        <param name="baud_rate">57600</param>
-        <param name="timeout_ms">1000</param>
-        <param name="step_enc_counts_per_rev">100</param>
-        <param name="bldc_enc_counts_per_rev">3436</param>
-      </hardware>
-      <joint name="lower_arm_joint">
-        <command_interface name="position"/>
-        <state_interface name="position"/>
-      </joint>
-    </ros2_control>
+    </xacro:end_effector>
+    <!-- Lidar -->
+    <xacro:lidar parent_link="base_link">
+        <origin xyz="0.122 0 ${body_height}" rpy="0 0 0"/>
+    </xacro:lidar>
 </robot>
