Commit message: more hardware interface changes, urdf now has conditional to check if in sim or not

File: src/rushbott_common/rushbott_description/urdf/arm.urdf.xacro (robot description, xacro)
@@ -29,13 +29,15 @@
             </xacro:inertial_cuboid_with_pose>
         </link>
-        <!-- <ros2_control name='${arm_joint_name}' type='system'>
-            <hardware>
-                <plugin>gz_ros2_control/GazeboSimSystem</plugin>
-            </hardware>
-            <joint name='${arm_joint_name}'>
-                <command_interface name='position'/>
-                <state_interface name='position'/>
-            </joint>
-        </ros2_control> -->
+        <xacro:if is_sim="true">
+            <ros2_control name='${arm_joint_name}' type='system'>
+                <hardware>
+                    <plugin>gz_ros2_control/GazeboSimSystem</plugin>
+                </hardware>
+                <joint name='${arm_joint_name}'>
+                    <command_interface name='position'/>
+                    <state_interface name='position'/>
+                </joint>
+            </ros2_control>
+        </xacro:if>
     </xacro:macro>
     <!--Arm Link Mimic-->
@@ -94,4 +96,15 @@
             </xacro:inertial_cuboid_with_pose>
         </link>
+        <xacro:if is_sim="true">
+            <ros2_control name='${arm_joint_name}' type='system'>
+                <hardware>
+                    <plugin>gz_ros2_control/GazeboSimSystem</plugin>
+                </hardware>
+                <joint name='${arm_joint_name}'>
+                    <command_interface name='position'/>
+                    <state_interface name='position'/>
+                </joint>
+            </ros2_control>
+        </xacro:if>
     </xacro:macro>
 </robot>

File: src/rushbott_common/rushbott_description/urdf/lidar.urdf.xacro (robot description, xacro)
@@ -27,28 +27,30 @@
         </xacro:inertial_cylinder_with_pose>
     </link>
-    <gazebo reference="lidar">
-        <sensor name="lidar" type="gpu_lidar">
-            <gz_frame_id>lidar</gz_frame_id>
-            <always_on>true</always_on>
-            <visualize>true</visualize>
-            <update_rate>10</update_rate>
-            <topic>scan</topic>
-            <lidar>
-                <scan>
-                    <horizontal>
-                        <samples>360</samples>
-                        <min_angle>-3.14</min_angle>
-                        <max_angle>3.14</max_angle>
-                    </horizontal>
-                </scan>
-                <range>
-                    <min>0.3</min>
-                    <max>12</max>
-                    <resolution>0.01</resolution>
-                </range>
-            </lidar>
-            <plugin name="gz::sim::systems::Sensors" filename = "gz-sim-sensors-system"></plugin>
-        </sensor>
-    </gazebo>
+    <xacro:if is_sim="true">
+        <gazebo reference="lidar">
+            <sensor name="lidar" type="gpu_lidar">
+                <gz_frame_id>lidar</gz_frame_id>
+                <always_on>true</always_on>
+                <visualize>true</visualize>
+                <update_rate>10</update_rate>
+                <topic>scan</topic>
+                <lidar>
+                    <scan>
+                        <horizontal>
+                            <samples>360</samples>
+                            <min_angle>-3.14</min_angle>
+                            <max_angle>3.14</max_angle>
+                        </horizontal>
+                    </scan>
+                    <range>
+                        <min>0.3</min>
+                        <max>12</max>
+                        <resolution>0.01</resolution>
+                    </range>
+                </lidar>
+                <plugin name="gz::sim::systems::Sensors" filename = "gz-sim-sensors-system"></plugin>
+            </sensor>
+        </gazebo>
+    </xacro:if>
 </xacro:macro>
 </robot>

File: src/rushbott_common/rushbott_description/urdf/rushbott.urdf.xacro (robot description, xacro)
@@ -6,4 +6,6 @@
     <xacro:include filename='arm.urdf.xacro'/>
     <xacro:include filename='lidar.urdf.xacro'/>
+    <!-- Simulation Check-->
+    <xacro:property name='is_sim'               value='false' />
     <!-- Body Properties -->
     <xacro:property name='body_mass'               value='2.300' />
@@ -76,4 +78,38 @@
         </xacro:inertial_cuboid_with_pose>
     </link>
+    <!-- Wheels with servos
+    <xacro:wheel_with_servo name='front_left' parent_link='base_link'>
+        <origin xyz='${wheelbase/2} ${track_width/2} ${-wheel_depth+servo_height}' rpy='0 0 0'/>
+        <axis xyz='0 0 1'/>
+    </xacro:wheel_with_servo>
+    <xacro:wheel_with_servo name='front_right' parent_link='base_link'>
+        <origin xyz='${wheelbase/2} ${-track_width/2} ${-wheel_depth+servo_height}' rpy='0 0 ${pi}'/>
+        <axis xyz='0 0 -1'/>
+    </xacro:wheel_with_servo>
+    <xacro:wheel_with_servo name='rear_left' parent_link='base_link'>
+        <origin xyz='${-wheelbase/2} ${track_width/2} ${-wheel_depth+servo_height}' rpy='0 0 0'/>
+        <axis xyz='0 0 1'/>
+    </xacro:wheel_with_servo>
+    <xacro:wheel_with_servo name='rear_right' parent_link='base_link'>
+        <origin xyz='${-wheelbase/2} ${-track_width/2} ${-wheel_depth+servo_height}' rpy='0 0 ${pi}'/>
+        <axis xyz='0 0 -1'/>
+    </xacro:wheel_with_servo>
+    Wheels
+    <xacro:wheel name='mid_left' parent_link='base_link'>
+        <origin xyz='0 ${track_width/2} ${-wheel_depth}' rpy='${-pi/2} 0 0'/>
+        <axis xyz='0 0 1'/>
+    </xacro:wheel>
+    <xacro:wheel name='mid_right' parent_link='base_link'>
+        <origin xyz='0 ${-track_width/2} ${-wheel_depth}' rpy='${-pi/2} 0 ${pi}'/>
+        <axis xyz='0 0 -1'/>
+    </xacro:wheel> -->
+    <!-- Gazebo (make this conditional later on) -->
+    <xacro:if is_sim="true">
+        <gazebo>
+            <plugin filename='libgz_ros2_control-system.so' name='gz_ros2_control::GazeboSimROS2ControlPlugin'>
+                <parameters>$(find rushbott_control)/config/control.yaml</parameters>
+            </plugin>
+        </gazebo>
+    </xacro:if>
     <!-- Arm -->
     <xacro:arm_link name='lower_arm' parent_link='base_link' length='${lower_arm_length}' width='${lower_arm_width}' mass='${lower_arm_mass}' offset='0' mesh='${lower_arm_mesh}'>
@@ -100,18 +136,26 @@
         <origin xyz='${suction_base_length} 0 0' rpy='0 0 0'/>
     </xacro:end_effector> -->
-    <ros2_control name="rushbott_control" type="system">
-      <hardware>
-        <plugin>rushbott_hardware/RoverSystemHardware</plugin>
-        <param name="loop_rate">30</param>
-        <param name="device">/dev/ttyACM0</param>
-        <param name="baud_rate">9600</param>
-        <param name="timeout_ms">2000</param>
-        <param name="step_enc_counts_per_rev">100</param>
-        <param name="bldc_enc_counts_per_rev">3436</param>
-      </hardware>
-      <joint name="lower_arm_joint">
-        <command_interface name="position"/>
-        <state_interface name="position"/>
-      </joint>
-    </ros2_control>
+    <!-- Lidar
+    <xacro:lidar parent_link="base_link">
+        <origin xyz="0.122 0 ${body_height}" rpy="0 0 0"/>
+    </xacro:lidar> -->
+    <xacro:if is_sim="false">
+        <ros2_control name="rushbott_control" type="system">
+        <hardware>
+            <plugin>rushbott_hardware/RoverSystemHardware</plugin>
+            <param name="loop_rate">30</param>
+            <param name="device">/dev/ttyACM0</param>
+            <param name="baud_rate">9600</param>
+            <param name="msg_attempts">6</param>
+            <param name="timeout_ms">300</param>
+            <param name="stepper_enc_per_rev">4096</param>
+            <param name="stepper_step_per_rev">800</param>
+            <param name="bldc_enc_per_rev">0</param>
+        </hardware>
+        <joint name="lower_arm_joint">
+            <command_interface name="position"/>
+            <state_interface name="position"/>
+        </joint>
+        </ros2_control>
+    </xacro:if>
 </robot>

File: src/rushbott_common/rushbott_description/urdf/wheel.urdf.xacro (robot description, xacro)
@@ -29,20 +29,22 @@
         <xacro:inertial_cylinder mass='${wheel_mass}' radius='${wheel_radius}' length='${wheel_width}'/>
     </link>
-    <ros2_control name='${wheel_joint_name}' type='system'>
-        <hardware>
-            <plugin>gz_ros2_control/GazeboSimSystem</plugin>
-        </hardware>
-        <joint name='${wheel_joint_name}'>
-            <command_interface name='velocity'/>
-            <state_interface name='position'/>
-        </joint>
-    </ros2_control>
-    <gazebo reference='${wheel_link_name}'>
-        <mu1 value="1.0"/>
-        <mu2 value="1.0"/>
-        <kp value="1.0"/>
-        <kd value="1.0"/>
-        <fdir1 value="1 0 0"/>
-    </gazebo>
+    <xacro:if is_sim="true">
+        <ros2_control name='${wheel_joint_name}' type='system'>
+            <hardware>
+                <plugin>gz_ros2_control/GazeboSimSystem</plugin>
+            </hardware>
+            <joint name='${wheel_joint_name}'>
+                <command_interface name='velocity'/>
+                <state_interface name='position'/>
+            </joint>
+        </ros2_control>
+        <gazebo reference='${wheel_link_name}'>
+            <mu1 value="1.0"/>
+            <mu2 value="1.0"/>
+            <kp value="1.0"/>
+            <kd value="1.0"/>
+            <fdir1 value="1 0 0"/>
+        </gazebo>
+    </xacro:if>
 </xacro:macro>
 </robot>

File: src/rushbott_common/rushbott_description/urdf/wheel_with_servo.urdf.xacro (robot description, xacro)
@@ -31,4 +31,5 @@
             <xacro:inertial_cylinder mass='${servo_mass}' radius='${servo_radius}' length='${servo_width}'/>
         </link>
+    <xacro:if is_sim="true">
         <ros2_control name='${servo_joint_name}' type='system'>
             <hardware>
@@ -43,4 +44,5 @@
             <xacro:insert_block name='axis'/>
         </xacro:wheel>
+    </xacro:if>
     </xacro:macro>
 </robot>

Commit message: Fixed issue where bullet-featherstone engine would cause rover to skid in Gazebo. Added conditionals to choose between simulated and real rover

File: src/rushbott_common/rushbott_description/urdf/arm.urdf.xacro (robot description, xacro)
@@ -10,4 +10,5 @@
             <xacro:insert_block name='limit'/>
             <axis xyz='0 1 0'/>
+            <dynamics damping="0.1" friction="0.2"/>
         </joint>
         <link name='${name}'>
@@ -29,5 +30,5 @@
             </xacro:inertial_cuboid_with_pose>
         </link>
-        <xacro:if is_sim="true">
+        <xacro:if value="${is_sim == True}">
             <ros2_control name='${arm_joint_name}' type='system'>
                 <hardware>
@@ -50,4 +51,5 @@
             <xacro:insert_block name='mimic'/>
             <axis xyz='0 1 0'/>
+            <dynamics damping="0.1" friction="0.2"/>
         </joint>
         <link name='${name}'>
@@ -96,15 +98,4 @@
             </xacro:inertial_cuboid_with_pose>
         </link>
-        <xacro:if is_sim="true">
-            <ros2_control name='${arm_joint_name}' type='system'>
-                <hardware>
-                    <plugin>gz_ros2_control/GazeboSimSystem</plugin>
-                </hardware>
-                <joint name='${arm_joint_name}'>
-                    <command_interface name='position'/>
-                    <state_interface name='position'/>
-                </joint>
-            </ros2_control>
-        </xacro:if>
     </xacro:macro>
 </robot>

File: src/rushbott_common/rushbott_description/urdf/lidar.urdf.xacro (robot description, xacro)
@@ -27,5 +27,5 @@
         </xacro:inertial_cylinder_with_pose>
     </link>
-    <xacro:if is_sim="true">
+    <xacro:if value="${is_sim == True}">
         <gazebo reference="lidar">
             <sensor name="lidar" type="gpu_lidar">

File: src/rushbott_common/rushbott_description/urdf/rushbott.urdf.xacro (robot description, xacro)
@@ -7,5 +7,5 @@
     <xacro:include filename='lidar.urdf.xacro'/>
     <!-- Simulation Check-->
-    <xacro:property name='is_sim'               value='false' />
+    <xacro:property name='is_sim'               value='true' />
     <!-- Body Properties -->
     <xacro:property name='body_mass'               value='2.300' />
@@ -78,5 +78,5 @@
         </xacro:inertial_cuboid_with_pose>
     </link>
-    <!-- Wheels with servos
+    <!-- Wheels with servos -->
     <xacro:wheel_with_servo name='front_left' parent_link='base_link'>
         <origin xyz='${wheelbase/2} ${track_width/2} ${-wheel_depth+servo_height}' rpy='0 0 0'/>
@@ -95,5 +95,5 @@
         <axis xyz='0 0 -1'/>
     </xacro:wheel_with_servo>
-    Wheels
+    <!-- Wheels -->
     <xacro:wheel name='mid_left' parent_link='base_link'>
         <origin xyz='0 ${track_width/2} ${-wheel_depth}' rpy='${-pi/2} 0 0'/>
@@ -103,13 +103,5 @@
         <origin xyz='0 ${-track_width/2} ${-wheel_depth}' rpy='${-pi/2} 0 ${pi}'/>
         <axis xyz='0 0 -1'/>
-    </xacro:wheel> -->
-    <!-- Gazebo (make this conditional later on) -->
-    <xacro:if is_sim="true">
-        <gazebo>
-            <plugin filename='libgz_ros2_control-system.so' name='gz_ros2_control::GazeboSimROS2ControlPlugin'>
-                <parameters>$(find rushbott_control)/config/control.yaml</parameters>
-            </plugin>
-        </gazebo>
-    </xacro:if>
+    </xacro:wheel>
     <!-- Arm -->
     <xacro:arm_link name='lower_arm' parent_link='base_link' length='${lower_arm_length}' width='${lower_arm_width}' mass='${lower_arm_mass}' offset='0' mesh='${lower_arm_mesh}'>
@@ -117,5 +109,5 @@
         <limit lower='${0.3}' upper='${pi-0.3}' effort='10' velocity='10'/>
     </xacro:arm_link>
-    <!-- <xacro:arm_link name='upper_arm' parent_link='lower_arm' length='${upper_arm_length}' width='${upper_arm_width}' mass='${upper_arm_mass}' offset='${upper_control_length}' mesh='${upper_arm_mesh}'>
+    <xacro:arm_link name='upper_arm' parent_link='lower_arm' length='${upper_arm_length}' width='${upper_arm_width}' mass='${upper_arm_mass}' offset='${upper_control_length}' mesh='${upper_arm_mesh}'>
         <origin xyz='${-lower_arm_length} 0 0' rpy='0 0 0'/>
         <limit lower='${-pi+0.3}' upper='${-0.3}' effort='10' velocity='10'/>
@@ -135,10 +127,10 @@
     <xacro:end_effector name='suction_head' parent_link='suction_base' length='${suction_head_length}' width='${suction_head_width}' mass='${suction_head_mass}' mesh='${suction_head_mesh}'>
         <origin xyz='${suction_base_length} 0 0' rpy='0 0 0'/>
-    </xacro:end_effector> -->
-    <!-- Lidar
+    </xacro:end_effector>
+    <!-- Lidar -->
     <xacro:lidar parent_link="base_link">
         <origin xyz="0.122 0 ${body_height}" rpy="0 0 0"/>
-    </xacro:lidar> -->
-    <xacro:if is_sim="false">
+    </xacro:lidar>
+    <xacro:if value="${is_sim == False}">
         <ros2_control name="rushbott_control" type="system">
         <hardware>
@@ -159,3 +151,11 @@
         </ros2_control>
     </xacro:if>
+        <!-- Gazebo (make this conditional later on) -->
+    <xacro:if value="${is_sim == True}">
+        <gazebo>
+            <plugin filename='libgz_ros2_control-system.so' name='gz_ros2_control::GazeboSimROS2ControlPlugin'>
+                <parameters>$(find rushbott_control)/config/control.yaml</parameters>
+            </plugin>
+        </gazebo>
+    </xacro:if>
 </robot>

File: src/rushbott_common/rushbott_description/urdf/wheel.urdf.xacro (robot description, xacro)
@@ -12,4 +12,5 @@
         <xacro:insert_block name='origin'/>
         <xacro:insert_block name='axis'/>
+        <dynamics damping="0.1" friction="0.2"/>
     </joint>
     <link name='${wheel_link_name}'>
@@ -29,5 +30,5 @@
         <xacro:inertial_cylinder mass='${wheel_mass}' radius='${wheel_radius}' length='${wheel_width}'/>
     </link>
-    <xacro:if is_sim="true">
+    <xacro:if value="${is_sim == True}">
         <ros2_control name='${wheel_joint_name}' type='system'>
             <hardware>
@@ -45,4 +46,13 @@
             <kd value="1.0"/>
             <fdir1 value="1 0 0"/>
+            <collision name="${wheel_link_name}_collision">
+                <surface>
+                    <friction>
+                        <torsional>
+                            <coefficient>0.0</coefficient>
+                        </torsional>
+                    </friction>
+                </surface>
+            </collision>
         </gazebo>
     </xacro:if>

File: src/rushbott_common/rushbott_description/urdf/wheel_with_servo.urdf.xacro (robot description, xacro)
@@ -14,4 +14,5 @@
             <axis xyz='0 0 -1'/>
             <limit lower = "${-pi/2}" upper = "${pi/2}" effort='10' velocity='10'/>
+            <dynamics damping="0.1" friction="0.2"/>
         </joint>
         <link name='${servo_link_name}'>
@@ -31,18 +32,18 @@
             <xacro:inertial_cylinder mass='${servo_mass}' radius='${servo_radius}' length='${servo_width}'/>
         </link>
-    <xacro:if is_sim="true">
-        <ros2_control name='${servo_joint_name}' type='system'>
-            <hardware>
-                <plugin>gz_ros2_control/GazeboSimSystem</plugin>
-            </hardware>
-            <joint name='${servo_joint_name}'>
-                <command_interface name='position'/>
-            </joint>
-        </ros2_control>
         <xacro:wheel name='${name}' parent_link='${servo_link_name}'>
             <origin xyz='0 0 ${-servo_height}' rpy='${-pi/2} 0 0'/>
             <xacro:insert_block name='axis'/>
         </xacro:wheel>
-    </xacro:if>
+        <xacro:if value="${is_sim == True}">
+            <ros2_control name='${servo_joint_name}' type='system'>
+                <hardware>
+                    <plugin>gz_ros2_control/GazeboSimSystem</plugin>
+                </hardware>
+                <joint name='${servo_joint_name}'>
+                    <command_interface name='position'/>
+                </joint>
+            </ros2_control>
+        </xacro:if>
     </xacro:macro>
 </robot>
