Commit message: real arm moves!

File: src/rushbott_common/rushbott_description/urdf/arm.urdf.xacro (robot description, xacro)
@@ -2,5 +2,5 @@
 <robot xmlns:xacro='http://www.ros.org/wiki/xacro'>
     <!--Arm Link-->
-    <xacro:macro name='arm_link' params='name parent_link length width offset mass mesh *origin *limit'>
+    <xacro:macro name='arm_link' params='name is_fake parent_link length width offset mass mesh *origin *limit'>
         <xacro:property name='arm_joint_name' value='${name}_joint'/>
         <joint name='${arm_joint_name}' type='revolute'>
@@ -34,4 +34,15 @@
                 <hardware>
                     <plugin>gz_ros2_control/GazeboSimSystem</plugin>
+                </hardware>
+                <joint name='${arm_joint_name}'>
+                    <command_interface name='position'/>
+                    <state_interface name='position'/>
+                </joint>
+            </ros2_control>
+        </xacro:if>
+        <xacro:if value="${is_fake == True and is_sim == False}">
+            <ros2_control name='${arm_joint_name}' type='system'>
+                <hardware>
+                    <plugin>mock_components/GenericSystem</plugin>
                 </hardware>
                 <joint name='${arm_joint_name}'>

File: src/rushbott_common/rushbott_description/urdf/rushbott.urdf.xacro (robot description, xacro)
@@ -7,5 +7,5 @@
     <xacro:include filename='lidar.urdf.xacro'/>
     <!-- Simulation Check-->
-    <xacro:property name='is_sim'               value='true' />
+    <xacro:property name='is_sim'               value='True' />
     <!-- Body Properties -->
     <xacro:property name='body_mass'               value='2.300' />
@@ -105,12 +105,12 @@
     </xacro:wheel>
     <!-- Arm -->
-    <xacro:arm_link name='lower_arm' parent_link='base_link' length='${lower_arm_length}' width='${lower_arm_width}' mass='${lower_arm_mass}' offset='0' mesh='${lower_arm_mesh}'>
+    <xacro:arm_link name='lower_arm' is_fake='false' parent_link='base_link' length='${lower_arm_length}' width='${lower_arm_width}' mass='${lower_arm_mass}' offset='0' mesh='${lower_arm_mesh}'>
         <origin xyz='${arm_x_position} 0 ${arm_z_position}' rpy='0 0 0'/>
-        <limit lower='${0.3}' upper='${pi-0.3}' effort='10' velocity='10'/>
+        <limit lower='${26 * pi / 180}' upper='${pi-0.3}' effort='10' velocity='10'/>
     </xacro:arm_link>
-    <xacro:arm_link name='upper_arm' parent_link='lower_arm' length='${upper_arm_length}' width='${upper_arm_width}' mass='${upper_arm_mass}' offset='${upper_control_length}' mesh='${upper_arm_mesh}'>
+    <xacro:arm_link name='upper_arm' is_fake='false' parent_link='lower_arm' length='${upper_arm_length}' width='${upper_arm_width}' mass='${upper_arm_mass}' offset='${upper_control_length}' mesh='${upper_arm_mesh}'>
         <origin xyz='${-lower_arm_length} 0 0' rpy='0 0 0'/>
-        <limit lower='${-pi+0.3}' upper='${-0.3}' effort='10' velocity='10'/>
-    </xacro:arm_link>
+        <limit lower='${-pi+(21 * pi / 180)}' upper='${-(21 * pi / 180)}' effort='10' velocity='10'/>
+    </xacro:arm_link>w
     <xacro:arm_link_mimic name='upper_control' parent_link='lower_arm' length='${upper_control_length}' width='${upper_control_width}' mass='${upper_control_mass}' mesh='${upper_control_mesh}'>
         <origin xyz='0 0 0' rpy='0 0 0'/>
@@ -121,5 +121,5 @@
         <mimic joint='upper_control_joint' multiplier='-1.0'/>
     </xacro:arm_link_mimic>
-    <xacro:arm_link name='suction_base' parent_link='upper_arm' length='${suction_base_length}' width='${suction_base_width}' mass='${suction_base_mass}' offset='0' mesh='${suction_base_mesh}'>
+    <xacro:arm_link name='suction_base' is_fake='false' parent_link='upper_arm' length='${suction_base_length}' width='${suction_base_width}' mass='${suction_base_mass}' offset='0' mesh='${suction_base_mesh}'>
         <origin xyz='${-upper_control_length+upper_arm_length} 0 0' rpy='0 0 0'/>
         <limit lower='${-2*pi}' upper='${2*pi}' effort='10' velocity='10'/>
@@ -134,19 +134,26 @@
     <xacro:if value="${is_sim == False}">
         <ros2_control name="rushbott_control" type="system">
-        <hardware>
-            <plugin>rushbott_hardware/RoverSystemHardware</plugin>
-            <param name="loop_rate">30</param>
-            <param name="device">/dev/ttyACM0</param>
-            <param name="baud_rate">9600</param>
-            <param name="msg_attempts">6</param>
-            <param name="timeout_ms">300</param>
-            <param name="stepper_enc_per_rev">4096</param>
-            <param name="stepper_step_per_rev">800</param>
-            <param name="bldc_enc_per_rev">0</param>
-        </hardware>
-        <joint name="lower_arm_joint">
-            <command_interface name="position"/>
-            <state_interface name="position"/>
-        </joint>
+            <hardware>
+                <plugin>rushbott_hardware/RoverSystemHardware</plugin>
+                <param name="loop_rate">30</param>
+                <param name="device">/dev/ttyACM0</param>
+                <param name="baud_rate">9600</param>
+                <param name="msg_attempts">6</param>
+                <param name="timeout_ms">300</param>
+                <param name="stepper_lower_initial">28</param>
+                <param name="stepper_upper_initial">-28</param>
+                <param name="stepper_gear_ratio">3</param>
+                <param name="stepper_enc_per_rev">400</param>
+                <param name="stepper_step_per_rev">400</param>
+                <param name="bldc_enc_per_rev">0</param>
+            </hardware>
+            <joint name="lower_arm_joint">
+                <command_interface name="position"/>
+                <state_interface name="position"/>
+            </joint>
+            <joint name="upper_arm_joint">
+                <command_interface name="position"/>
+                <state_interface name="position"/>
+            </joint>
         </ros2_control>
     </xacro:if>

Commit message: fixed arm urdf angles to be follow convention, created joint group class to handle conversions between ros and arduino, added calibration functionality, fixed urdf parameters to work between sim and real robot

File: src/rushbott_common/rushbott_description/urdf/arm.urdf.xacro (robot description, xacro)
@@ -9,10 +9,10 @@
             <xacro:insert_block name='origin'/>
             <xacro:insert_block name='limit'/>
-            <axis xyz='0 1 0'/>
+            <axis xyz='0 0 1'/>
             <dynamics damping="0.1" friction="0.2"/>
         </joint>
         <link name='${name}'>
             <visual>
-                <origin xyz="0 0 0" rpy="${-pi/2} ${-pi} ${-pi/2}"/>
+                <origin xyz="0 0 0" rpy="0 ${pi/2} 0"/>
                 <geometry>
                     <mesh filename='${mesh}' scale='0.001 0.001 0.001'/>
@@ -21,14 +21,14 @@
             </visual>
             <collision>
-                <origin xyz='${offset-length/2} 0 0' rpy ='0 ${pi/2} 0'/>
+                <origin xyz='${length/2 - offset} 0 0' rpy ='0 0 0'/>
                 <geometry>
-                    <box size='${width} ${width} ${length}'/>
+                    <box size='${length} ${width} ${width}'/>
                 </geometry>
             </collision>
-            <xacro:inertial_cuboid_with_pose mass='${mass}' x='${width}' y='${width}' z='${length}'>
-                <origin xyz='${offset-length/2} 0 0' rpy='0 ${pi/2} 0'/>
+            <xacro:inertial_cuboid_with_pose mass='${mass}' x='${length}' y='${width}' z='${width}'>
+                <origin xyz='${length/2 - offset} 0 0' rpy='0 0 0'/>
             </xacro:inertial_cuboid_with_pose>
         </link>
-        <xacro:if value="${is_sim == True}">
+        <xacro:if value="$(arg is_sim)">
             <ros2_control name='${arm_joint_name}' type='system'>
                 <hardware>
@@ -37,53 +37,21 @@
                 <joint name='${arm_joint_name}'>
                     <command_interface name='position'/>
-                    <command_interface name="velocity"/>
                     <state_interface name='position'/>
-                    <state_interface name='velocity'/>
                 </joint>
             </ros2_control>
         </xacro:if>
-        <xacro:if value="${is_fake == True and is_sim == False}">
-            <ros2_control name='${arm_joint_name}' type='system'>
-                <hardware>
-                    <plugin>mock_components/GenericSystem</plugin>
-                </hardware>
-                <joint name='${arm_joint_name}'>
-                    <command_interface name='position'/>
-                    <command_interface name="velocity"/>
-                    <state_interface name='position'/>
-                    <state_interface name='velocity'/>
-                </joint>
-            </ros2_control>
+        <xacro:if value="${is_fake == True}">
+            <xacro:unless value="$(arg is_sim)">
+                <ros2_control name='${arm_joint_name}' type='system'>
+                    <hardware>
+                        <plugin>mock_components/GenericSystem</plugin>
+                    </hardware>
+                    <joint name='${arm_joint_name}'>
+                        <command_interface name='position'/>
+                        <state_interface name='position'/>
+                    </joint>
+                </ros2_control>
+            </xacro:unless>
         </xacro:if>
-    </xacro:macro>
-    <!--Arm Link Mimic-->
-    <xacro:macro name='arm_link_mimic' params='name parent_link length width mass mesh *origin *mimic'>
-        <xacro:property name='arm_joint_name' value='${name}_joint'/>
-        <joint name='${arm_joint_name}' type='continuous'>
-            <parent link='${parent_link}'/>
-            <child link='${name}'/>
-            <xacro:insert_block name='origin'/>
-            <xacro:insert_block name='mimic'/>
-            <axis xyz='0 1 0'/>
-            <dynamics damping="0.1" friction="0.2"/>
-        </joint>
-        <link name='${name}'>
-            <visual>
-                <origin xyz="0 0 0" rpy="${-pi/2} ${-pi} ${-pi/2}"/>
-                <geometry>
-                    <mesh filename='${mesh}' scale='0.001 0.001 0.001'/>
-                </geometry>
-                <xacro:insert_block name='material_orange'/>
-            </visual>
-            <collision>
-                <origin xyz='${-length/2} 0 0' rpy ='0 ${pi/2} 0'/>
-                <geometry>
-                    <box size='${width} ${width} ${length}'/>
-                </geometry>
-            </collision>
-            <xacro:inertial_cuboid_with_pose mass='${mass}' x='${width}' y='${width}' z='${length}'>
-                <origin xyz='${-length/2} 0 0' rpy='0 ${pi/2} 0'/>
-            </xacro:inertial_cuboid_with_pose>
-        </link>
     </xacro:macro>
      <!--End Effector-->
@@ -97,5 +65,5 @@
         <link name='${name}'>
             <visual>
-                <origin xyz="0 0 0" rpy="${-pi/2} ${-pi} ${-pi/2}"/>
+                <origin xyz="0 0 0" rpy="0 ${-pi/2} 0"/>
                 <geometry>
                     <mesh filename='${mesh}' scale='0.001 0.001 0.001'/>
@@ -104,11 +72,11 @@
             </visual>
             <collision>
-                <origin xyz='${length/2} 0 0' rpy ='0 ${pi/2} 0'/>
+                <origin xyz='${length/2} 0 0' rpy ='0 0 0'/>
                 <geometry>
-                    <box size='${width} ${width} ${length}'/>
+                    <box size='${length} ${width} ${width}'/>
                 </geometry>
             </collision>
-            <xacro:inertial_cuboid_with_pose mass='${mass}' x='${width}' y='${width}' z='${length}'>
-                <origin xyz='${length/2} 0 0' rpy='0 ${pi/2} 0'/>
+            <xacro:inertial_cuboid_with_pose mass='${mass}' x='${length}' y='${width}' z='${width}'>
+                <origin xyz='${length/2} 0 0' rpy='0 0 0'/>
             </xacro:inertial_cuboid_with_pose>
         </link>

File: src/rushbott_common/rushbott_description/urdf/lidar.urdf.xacro (robot description, xacro)
@@ -27,5 +27,5 @@
         </xacro:inertial_cylinder_with_pose>
     </link>
-    <xacro:if value="${is_sim == True}">
+    <xacro:if value="$(arg is_sim)">
         <gazebo reference="lidar">
             <sensor name="lidar" type="gpu_lidar">

File: src/rushbott_common/rushbott_description/urdf/rushbott.urdf.xacro (robot description, xacro)
@@ -6,6 +6,7 @@
     <xacro:include filename='arm.urdf.xacro'/>
     <xacro:include filename='lidar.urdf.xacro'/>
+    <xacro:include filename='ros2_control.urdf.xacro'/>
     <!-- Simulation Check-->
-    <xacro:property name='is_sim'               value='False' />
+    <xacro:arg name='is_sim'               default='False'/>
     <!-- Body Properties -->
     <xacro:property name='body_mass'               value='2.300' />
@@ -78,49 +79,41 @@
         </xacro:inertial_cuboid_with_pose>
     </link>
-    <xacro:if value="${is_sim == True}">
+    <xacro:if value="$(arg is_sim)">
         <!-- Wheels with servos -->
-        <xacro:wheel_with_servo name='front_left' parent_link='base_link'>
+        <xacro:wheel_with_servo name='front_left' is_fake='True' parent_link='base_link'>
             <origin xyz='${wheelbase/2} ${track_width/2} ${-wheel_depth+servo_height}' rpy='0 0 0'/>
             <axis xyz='0 0 1'/>
         </xacro:wheel_with_servo>
-        <xacro:wheel_with_servo name='front_right' parent_link='base_link'>
+        <xacro:wheel_with_servo name='front_right' is_fake='True' parent_link='base_link'>
             <origin xyz='${wheelbase/2} ${-track_width/2} ${-wheel_depth+servo_height}' rpy='0 0 ${pi}'/>
             <axis xyz='0 0 -1'/>
         </xacro:wheel_with_servo>
-        <xacro:wheel_with_servo name='rear_left' parent_link='base_link'>
+        <xacro:wheel_with_servo name='rear_left' is_fake='True' parent_link='base_link'>
             <origin xyz='${-wheelbase/2} ${track_width/2} ${-wheel_depth+servo_height}' rpy='0 0 0'/>
             <axis xyz='0 0 1'/>
         </xacro:wheel_with_servo>
-        <xacro:wheel_with_servo name='rear_right' parent_link='base_link'>
+        <xacro:wheel_with_servo name='rear_right' is_fake='True' parent_link='base_link'>
             <origin xyz='${-wheelbase/2} ${-track_width/2} ${-wheel_depth+servo_height}' rpy='0 0 ${pi}'/>
             <axis xyz='0 0 -1'/>
         </xacro:wheel_with_servo>
         <!-- Wheels -->
-        <xacro:wheel name='mid_left' parent_link='base_link'>
+        <xacro:wheel name='mid_left' is_fake='True' parent_link='base_link'>
             <origin xyz='0 ${track_width/2} ${-wheel_depth}' rpy='${-pi/2} 0 0'/>
             <axis xyz='0 0 1'/>
         </xacro:wheel>
-        <xacro:wheel name='mid_right' parent_link='base_link'>
+        <xacro:wheel name='mid_right' is_fake='True' parent_link='base_link'>
             <origin xyz='0 ${-track_width/2} ${-wheel_depth}' rpy='${-pi/2} 0 ${pi}'/>
             <axis xyz='0 0 -1'/>
         </xacro:wheel>
     </xacro:if>
-    <!-- Arm -->
+    <!-- Arm --> 40 - 155, -30, -150
     <xacro:arm_link name='lower_arm' is_fake='False' parent_link='base_link' length='${lower_arm_length}' width='${lower_arm_width}' mass='${lower_arm_mass}' offset='0' mesh='${lower_arm_mesh}'>
-        <origin xyz='${arm_x_position} 0 ${arm_z_position}' rpy='0 0 0'/>
-        <limit lower='${26 * pi / 180}' upper='${pi-0.3}' effort='10' velocity='10'/>
+        <origin xyz='${arm_x_position} 0 ${arm_z_position}' rpy='${pi/2} 0 0'/>
+        <limit lower='${40 * pi / 180}' upper='${155 * pi / 180}' effort='10' velocity='10'/>
     </xacro:arm_link>
     <xacro:arm_link name='upper_arm' is_fake='False' parent_link='lower_arm' length='${upper_arm_length}' width='${upper_arm_width}' mass='${upper_arm_mass}' offset='${upper_control_length}' mesh='${upper_arm_mesh}'>
-        <origin xyz='${-lower_arm_length} 0 0' rpy='0 0 0'/>
-        <limit lower='${-pi+(21 * pi / 180)}' upper='${-(21 * pi / 180)}' effort='10' velocity='10'/>
+        <origin xyz='${lower_arm_length} 0 0' rpy='0 0 0'/>
+        <limit lower='${-150 * pi / 180}' upper='${-30 * pi / 180}' effort='10' velocity='10'/>
     </xacro:arm_link>
-    <xacro:arm_link_mimic name='upper_control' parent_link='lower_arm' length='${upper_control_length}' width='${upper_control_width}' mass='${upper_control_mass}' mesh='${upper_control_mesh}'>
-        <origin xyz='0 0 0' rpy='0 0 0'/>
-        <mimic joint='upper_arm_joint' multiplier='1.0'/>
-    </xacro:arm_link_mimic>
-    <xacro:arm_link_mimic name='upper_link' parent_link='upper_control' length='${upper_link_length}' width='${upper_link_width}' mass='${upper_link_mass}' mesh='${upper_link_mesh}'>
-        <origin xyz='${-upper_control_length} 0 0' rpy='0 0 0'/>
-        <mimic joint='upper_control_joint' multiplier='-1.0'/>
-    </xacro:arm_link_mimic>
     <xacro:arm_link name='suction_base' is_fake='True' parent_link='upper_arm' length='${suction_base_length}' width='${suction_base_width}' mass='${suction_base_mass}' offset='0' mesh='${suction_base_mesh}'>
         <origin xyz='${-upper_control_length+upper_arm_length} 0 0' rpy='0 0 0'/>
@@ -134,36 +127,9 @@
         <origin xyz="0.122 0 ${body_height}" rpy="0 0 0"/>
     </xacro:lidar>
-    <xacro:if value="${is_sim == False}">
-        <ros2_control name="rushbott_control" type="system">
-            <hardware>
-                <plugin>rushbott_hardware/RoverSystemHardware</plugin>
-                <param name="loop_rate">30</param>
-                <param name="device">/dev/ttyACM0</param>
-                <param name="baud_rate">9600</param>
-                <param name="msg_attempts">10</param>
-                <param name="timeout_ms">200</param>
-                <param name="stepper_gear_ratio">3</param>
-                <param name="stepper_enc_per_rev">1600</param>
-                <param name="stepper_step_per_rev">1600</param>
-                <param name="bldc_enc_per_rev">0</param>
-            </hardware>
-            <joint name="lower_arm_joint">
-                <command_interface name="position"/>
-                <command_interface name="velocity"/>
-                <state_interface name="position"/>
-                <state_interface name="velocity"/>
-                <param name="initial_value">0.3</param>
-            </joint>
-            <joint name="upper_arm_joint">
-                <command_interface name="position"/>
-                <command_interface name="velocity"/>
-                <state_interface name="position"/>
-                <state_interface name="velocity"/>
-                <param name="initial_value">-0.3</param>
-            </joint>
-        </ros2_control>
-    </xacro:if>
+    <xacro:unless value="$(arg is_sim)">
+        <xacro:ros2_control/>
+    </xacro:unless>
         <!-- Gazebo (make this conditional later on) -->
-    <xacro:if value="${is_sim == True}">
+    <xacro:if value="$(arg is_sim)">
         <gazebo>
             <plugin filename='libgz_ros2_control-system.so' name='gz_ros2_control::GazeboSimROS2ControlPlugin'>

File: src/rushbott_common/rushbott_description/urdf/wheel.urdf.xacro (robot description, xacro)
@@ -1,5 +1,5 @@
 <?xml version='1.0'?>
 <robot xmlns:xacro='http://www.ros.org/wiki/xacro'>
-<xacro:macro name='wheel' params='name parent_link *origin *axis'>
+<xacro:macro name='wheel' params='name is_fake parent_link *origin *axis'>
     <xacro:property name='wheel_link_name'  value='${name}_wheel'/>
     <xacro:property name='wheel_joint_name' value='${wheel_link_name}_joint'/>
@@ -30,5 +30,18 @@
         <xacro:inertial_cylinder mass='${wheel_mass}' radius='${wheel_radius}' length='${wheel_width}'/>
     </link>
-    <xacro:if value="${is_sim == True}">
+    <xacro:if value="${is_fake == True}">
+        <xacro:unless value="$(arg is_sim)">
+            <ros2_control name='${wheel_joint_name}' type='system'>
+                <hardware>
+                    <plugin>mock_components/GenericSystem</plugin>
+                </hardware>
+                <joint name='${wheel_joint_name}'>
+                    <command_interface name='velocity'/>
+                    <state_interface name='position'/>
+                </joint>
+            </ros2_control>
+        </xacro:unless>
+    </xacro:if>
+    <xacro:if value="$(arg is_sim)">
         <ros2_control name='${wheel_joint_name}' type='system'>
             <hardware>

File: src/rushbott_common/rushbott_description/urdf/wheel_with_servo.urdf.xacro (robot description, xacro)
@@ -2,5 +2,5 @@
 <robot xmlns:xacro='http://www.ros.org/wiki/xacro'>
     <xacro:include filename='wheel.urdf.xacro'/>
-    <xacro:macro name='wheel_with_servo' params='name parent_link *origin *axis'>
+    <xacro:macro name='wheel_with_servo' params='name is_fake parent_link *origin *axis'>
         <xacro:property name='servo_link_name'  value='${name}_servo'/>
         <xacro:property name='servo_joint_name' value='${servo_link_name}_joint'/>
@@ -32,9 +32,21 @@
             <xacro:inertial_cylinder mass='${servo_mass}' radius='${servo_radius}' length='${servo_width}'/>
         </link>
-        <xacro:wheel name='${name}' parent_link='${servo_link_name}'>
+        <xacro:wheel name='${name}' is_fake='${is_fake}' parent_link='${servo_link_name}'>
             <origin xyz='0 0 ${-servo_height}' rpy='${-pi/2} 0 0'/>
             <xacro:insert_block name='axis'/>
         </xacro:wheel>
-        <xacro:if value="${is_sim == True}">
+        <xacro:if value="${is_fake == True}">
+            <xacro:unless value="$(arg is_sim)">
+                <ros2_control name='${servo_joint_name}' type='system'>
+                    <hardware>
+                        <plugin>mock_components/GenericSystem</plugin>
+                    </hardware>
+                    <joint name='${servo_joint_name}'>
+                        <command_interface name='position'/>
+                    </joint>
+                </ros2_control>
+            </xacro:unless>
+        </xacro:if>
+        <xacro:if value="$(arg is_sim)">
             <ros2_control name='${servo_joint_name}' type='system'>
                 <hardware>
